File: placas/Esp32Version/Esp32Version.kicad_pcb (KiCad board)
At the start: 2 copper layers, 21 parts, among them J1 Conn_01x04_Male, J2 Conn_01x04_Male, J3 Conn_01x04_Male, J4 Conn_01x04_Male, J6 Conn_01x08_Female, SW2 SW_DPDT_x2

Commit message: chg
Parts:
- added BOLITA: BolitaHolder, propios:BolitaHolder, F.Cu at (102.0, 8.00)
- added HOLDER: SharpHolder, propios:SharpHolder, F.Cu at (70.5, 41.8)
- added HOLDER: SharpHolder, propios:SharpHolder, F.Cu at (133.0, 41.7)
- added HOLDER: SharpHolder, propios:SharpHolder, F.Cu at (101.6, 23.9)
- added REF**: MotorHolder, propios:MotorHolder, F.Cu at (50.5, 123.3)
- added REF**: MotorHolder, propios:MotorHolder, F.Cu at (130.1, 123.0)
- moved On Led 31.6 mm to (133.9, 62.7), turned to 180 degrees
- moved R2 12.2 mm to (131.3, 78.0), turned to 90 degrees
- moved Step Up 10.8 mm to (155.9, 97.5)
- moved CNY70 10.6 mm to (128.2, 23.0)
- moved SHARP_C 4.11 mm to (96.3, 45.0)
- moved MPU6050 2.51 mm to (65.3, 75.9)
- renumbered J1 to CNY70, J6 to MPU6050, J3 to SHARP_C, J4 to SHARP_D, J2 to SHARP_I
Routing:
- net /Vin: track 123.7 -> 72.6 mm
- net /CNY70: track 215.0 -> 253.7 mm
- net GND: track 220.6 -> 209.9 mm
- net /SHARP_A: track 19.7 -> 15.6 mm
- net /VOUT: track 63.5 -> 61.3 mm
- net /3,3v: track 487.7 -> 489.2 mm
- net /SCL: track 27.5 -> 26.1 mm
- net /SDA: track 39.4 -> 38.0 mm
- net Net-(D4-Pad2): track 6.22 -> 5.08 mm
Other:
- board text added: "D - +"
