File: placas/Laberinto/Esp32Version/Esp32Version.kicad_sch (KiCad schematic)
At the start: 21 parts, among them J1 Conn_01x02_Male, J2 Conn_01x06_Male, J3 Conn_01x06_Male, J4 Conn_01x04_Male, J5 Conn_01x04_Male, J6 Conn_01x04_Male, J7 Conn_01x04_Male, J8 Conn_01x08_Female, SW1 SW_Push, SW2 SW_Push, SW3 SW_DPDT_x2, SW4 SW_Push, U1 ESP32-Devkit-V1, U2 tb6612fng, U3 Mt3608

Commit message: SDF
Parts:
- R3: value R -> (none); footprint Resistor_THT:R_Axial_DIN0207_L6.3mm_D2.5mm_P10.16mm_Horizontal -> (none)
Changed lines of the file:
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@@
       (effects (font (size 1.27 1.27)) (justify left))
     )
-    (property "Value" "R" (id 1) (at 60.706 131.5719 0)
+    (property "Value" "" (id 1) (at 60.706 131.5719 0)
       (effects (font (size 1.27 1.27)) (justify left))
     )
-    (property "Footprint" "Resistor_THT:R_Axial_DIN0207_L6.3mm_D2.5mm_P10.16mm_Horizontal" (id 2) (at 57.15 130.302 90)
+    (property "Footprint" "" (id 2) (at 57.15 130.302 90)
       (effects (font (size 1.27 1.27)) hide)
     )
