File: placas/Laberinto/Esp32Version/Esp32Version.kicad_pcb (KiCad board)
At the start: 2 copper layers, 27 parts, among them SW2 SW_DPDT_x2

Commit message: 234
Routing:
- net /VOUT: track 61.3 -> 82.4 mm
Changed lines of the file:
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@@
+  )
+  (dimension (type aligned) (layer "B.Cu")
+    (pts (xy 47.244 19.05) (xy 156.464 18.32))
+    (height -4.349902)
+    (gr_text "109,2224 mm" (at 101.812897 12.535235 0.3829453968) (layer "B.Cu")
+      (effects (font (size 1.5 1.5) (thickness 0.3)))
+    )
+    (format (units 3) (units_format 1) (precision 4))
+    (style (thickness 0.2) (arrow_length 1.27) (text_position_mode 0) (extension_height 0.58642) (extension_offset 0.5) keep_text_aligned)
   )
   (dimension (type aligned) (layer "B.Cu")
@@
     (height 6.770012)
     (gr_text "13,5580 mm" (at 53.802452 43.163003 -0.1098752354) (layer "B.Cu")
+      (effects (font (size 1.5 1.5) (thickness 0.3)))
+    )
+    (format (units 3) (units_format 1) (precision 4))
+    (style (thickness 0.2) (arrow_length 1.27) (text_position_mode 0) (extension_height 0.58642) (extension_offset 0.5) keep_text_aligned)
+  )
+  (dimension (type aligned) (layer "B.Cu")
+    (pts (xy 46.736 140.716) (xy 46.99 18.32))
+    (height -28.951787)
+    (gr_text "122,3963 mm" (at 16.111279 79.454183 89.88109818) (layer "B.Cu")
       (effects (font (size 1.5 1.5) (thickness 0.3)))
     )
@@
   (segment (start 101.348 116.84) (end 101.348 105.918) (width 1) (layer "B.Cu") (net 10))
   (segment (start 109.474 116.84) (end 101.348 116.84) (width 1) (layer "B.Cu") (net 10))
+  (segment (start 123.636 96.636) (end 125 98) (width 1) (layer "B.Cu") (net 11))
   (segment (start 118.364 93.472) (end 121.797585 93.472) (width 1) (layer "B.Cu") (net 11))
   (segment (start 109.474 119.38) (end 93.98 119.38) (width 1) (layer "B.Cu") (net 11))
-  (segment (start 118.364 105.41) (end 118.364 93.472) (width 1) (layer "B.Cu") (net 11))
-  (segment (start 109.474 119.38) (end 118.364 119.38) (width 1) (layer "B.Cu") (net 11))
   (segment (start 117.856 105.918) (end 111.508 105.918) (width 1) (layer "B.Cu") (net 11))
   (segment (start 121.797585 93.472) (end 121.9245 93.598915) (width 1) (layer "B.Cu") (net 11))
-  (segment (start 118.364 119.38) (end 118.364 105.41) (width 1) (layer "B.Cu") (net 11))
+  (segment (start 118.364 96.636) (end 118.364 93.472) (width 1) (layer "B.Cu") (net 11))
+  (segment (start 124.62 119.38) (end 109.474 119.38) (width 1) (layer "B.Cu") (net 11))
+  (segment (start 118.364 96.636) (end 123.636 96.636) (width 1) (layer "B.Cu") (net 11))
   (segment (start 93.98 119.38) (end 93.726 119.126) (width 1) (layer "B.Cu") (net 11))
+  (segment (start 118.364 105.41) (end 118.364 96.636) (width 1) (layer "B.Cu") (net 11))
+  (segment (start 125 119) (end 124.62 119.38) (width 1) (layer "B.Cu") (net 11))
   (segment (start 118.364 105.41) (end 117.856 105.918) (width 1) (layer "B.Cu") (net 11))
+  (segment (start 125 98) (end 125 119) (width 1) (layer "B.Cu") (net 11))
   (segment (start 109.474 121.92) (end 97.282 121.92) (width 1) (layer "B.Cu") (net 12))
   (segment (start 86.36 128.524) (end 85.979 128.143) (width 1) (layer "B.Cu") (net 12))
