File: placas/Laberinto/BluePillVersion/BluePillVersion/BluePillVersion.kicad_pcb (KiCad board)
At the start: 2 copper layers, 23 parts, among them J1 Conn_01x04_Male, J2 Conn_01x04_Male, J3 Conn_01x04_Male, J4 Conn_01x04_Male, J5 Conn_01x06_Female, J6 Conn_01x06_Female, J7 Conn_01x02_Male, J8 Conn_01x08_Female, SW1 SW_Push, SW2 SW_DPDT_x2, SW3 SW_Push, SW4 SW_Push, U1 YAAJ_BluePill_Part_Like_SWD_B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, U2 tb6612fng, U3 Mt3608

Commit message: 234
Parts:
- moved J4 2.86 mm to (155.9, 59.4)
