File: placas/Laberinto/BluePill/Modularizado/BluePillVersion/Placa_Motores_sch.kicad_sch (KiCad schematic)
At the start: 4 parts, among them J1 Conn_01x06_Female, J2 Conn_01x06_Female, U1 tb6612fng, U2 Mt3608

Commit message: gh
Parts:
- added J12, J13: Conn_01x04_Male, symbol Connector:Conn_01x04_Male
- added J14: (no value), symbol Connector:Conn_01x08_Male
Connections:
- net 5v: now also J12.2 (Pin_2)
- net AIN1: now also J14.3 (Pin_3)
- net AIN2: now also J14.2 (Pin_2)
- net BIN1: now also J14.5 (Pin_5)
- net BIN2: now also J14.6 (Pin_6)
- net GND: now also J12.1 (Pin_1), J12.4 (Pin_4), J14.8 (Pin_8)
- net MA1: now also J13.4 (Pin_4)
- net MA2: now also J13.3 (Pin_3)
- net MB1: now also J13.2 (Pin_2)
- net MB2: now also J13.1 (Pin_1)
- net PWMA: now also J14.1 (Pin_1)
- net PWMB: now also J14.7 (Pin_7)
- net STBY: now also J14.4 (Pin_4)
- net VIn: now also J12.3 (Pin_3)
Other:
- note added: "conetores"
Changed lines of the file:
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@@
+    (stroke (width 0) (type default) (color 0 0 0 0))
+  )
+  (polyline (pts (xy 12.954 67.564) (xy 61.722 67.564))
     (stroke (width 0) (type default) (color 0 0 0 0))
   )
@@
     (stroke (width 0) (type default) (color 0 0 0 0))
   )
+  (polyline (pts (xy 61.722 67.564) (xy 61.722 103.378))
+    (stroke (width 0) (type default) (color 0 0 0 0))
+  )
   (wire (pts (xy 48.768 64.262) (xy 22.098 64.262))
     (stroke (width 0) (type default) (color 0 0 0 0))
@@
     (stroke (width 0) (type default) (color 0 0 0 0))
   )
+  (wire (pts (xy 32.004 73.406) (xy 29.718 73.406))
+    (stroke (width 0) (type default) (color 0 0 0 0))
+  )
   (polyline (pts (xy 62.992 12.954) (xy 62.992 44.45))
     (stroke (width 0) (type default) (color 0 0 0 0))
@@
     (stroke (width 0) (type default) (color 0 0 0 0))
   )
+  (wire (pts (xy 32.004 81.026) (xy 29.718 81.026))
+    (stroke (width 0) (type default) (color 0 0 0 0))
+  )
   (wire (pts (xy 22.098 60.452) (xy 23.368 60.452))
     (stroke (width 0) (type default) (color 0 0 0 0))
@@
     (stroke (width 0) (type default) (color 0 0 0 0))
   )
+  (polyline (pts (xy 61.722 103.378) (xy 12.954 103.378))
+    (stroke (width 0) (type default) (color 0 0 0 0))
+  )
   (wire (pts (xy 22.098 64.262) (xy 22.098 60.452))
     (stroke (width 0) (type default) (color 0 0 0 0))
@@
     (stroke (width 0) (type default) (color 0 0 0 0))
   )
+  (polyline (pts (xy 12.954 103.378) (xy 12.954 67.564))
+    (stroke (width 0) (type default) (color 0 0 0 0))
+  )
   (text "Motors\n" (at 54.864 33.274 0)
     (effects (font (size 1.27 1.27)) (justify left bottom))
   )
+  (text "conetores\n" (at 51.816 103.124 0)
+    (effects (font (size 1.27 1.27)) (justify left bottom))
+  )
   (text "Motor Driver\n" (at 49.53 66.294 0)
     (effects (font (size 1.27 1.27)) (justify left bottom))
@@
     (effects (font (size 1.27 1.27)) (justify left bottom))
   )
+  (label "AIN1" (at 48.514 79.756 0)
+    (effects (font (size 1.27 1.27)) (justify left bottom))
+  )
+  (label "MB1" (at 29.972 90.17 0)
+    (effects (font (size 1.27 1.27)) (justify left bottom))
+  )
   (label "AO1" (at 48.768 50.292 0)
     (effects (font (size 1.27 1.27)) (justify left bottom))
@@
     (effects (font (size 1.27 1.27)) (justify right bottom))
   )
+  (label "BIN2" (at 48.514 87.376 0)
+    (effects (font (size 1.27 1.27)) (justify left bottom))
+  )
   (label "VOut" (at 103.632 22.606 0)
     (effects (font (size 1.27 1.27)) (justify left bottom))
   )
+  (label "MB2" (at 29.972 87.63 0)
+    (effects (font (size 1.27 1.27)) (justify left bottom))
+  )
+  (label "BIN1" (at 48.514 84.836 0)
+    (effects (font (size 1.27 1.27)) (justify left bottom))
+  )
   (label "BO2" (at 48.768 55.372 0)
     (effects (font (size 1.27 1.27)) (justify left bottom))
   )
+  (label "PWMB" (at 48.514 89.916 0)
+    (effects (font (size 1.27 1.27)) (justify left bottom))
+  )
   (label "VIn" (at 72.898 22.606 180)
     (effects (font (size 1.27 1.27)) (justify right bottom))
   )
+  (label "AIN2" (at 48.514 77.216 0)
+    (effects (font (size 1.27 1.27)) (justify left bottom))
+  )
+  (label "MA1" (at 29.972 95.25 0)
+    (effects (font (size 1.27 1.27)) (justify left bottom))
+  )
   (label "VOut" (at 48.768 42.672 0)
     (effects (font (size 1.27 1.27)) (justify left bottom))
   )
+  (label "MA2" (at 29.972 92.71 0)
+    (effects (font (size 1.27 1.27)) (justify left bottom))
+  )
+  (label "STBY" (at 48.514 82.296 0)
+    (effects (font (size 1.27 1.27)) (justify left bottom))
+  )
   (label "5v" (at 48.768 45.212 0)
     (effects (font (size 1.27 1.27)) (justify left bottom))
@@
     (effects (font (size 1.27 1.27)) (justify right bottom))
   )
+  (label "PWMA" (at 48.514 74.676 0)
+    (effects (font (size 1.27 1.27)) (justify left bottom))
+  )
   (label "AO2" (at 48.768 52.832 0)
     (effects (font (size 1.27 1.27)) (justify left bottom))
@@
     (effects (font (size 1.27 1.27)) (justify right bottom))
   )
+  (label "VIn" (at 29.718 78.486 0)
+    (effects (font (size 1.27 1.27)) (justify left bottom))
+  )
   (label "STBY" (at 23.368 50.292 180)
     (effects (font (size 1.27 1.27)) (justify right bottom))
@@
     (effects (font (size 1.27 1.27)) (justify right bottom))
   )
+  (label "5v" (at 29.718 75.946 0)
+    (effects (font (size 1.27 1.27)) (justify left bottom))
+  )
   (label "MA2" (at 33.528 23.368 270)
     (effects (font (size 1.27 1.27)) (justify right bottom))
+  )
+  (symbol (lib_id "power:GND") (at 32.004 73.406 90) (unit 1)
+    (in_bom yes) (on_board yes) (fields_autoplaced)
+    (property "Reference" "#PWR0122" (id 0) (at 38.354 73.406 0)
+      (effects (font (size 1.27 1.27)) hide)
+    )
+    (property "Value" "GND" (id 1) (at 35.179 73.8398 90)
+      (effects (font (size 1.27 1.27)) (justify right))
+    )
+    (property "Footprint" "" (id 2) (at 32.004 73.406 0)
+      (effects (font (size 1.27 1.27)) hide)
+    )
+    (property "Datasheet" "" (id 3) (at 32.004 73.406 0)
+      (effects (font (size 1.27 1.27)) hide)
+    )
+    (pin "1")
   )
   (symbol (lib_id "propios:tb6612fng") (at 36.068 37.592 0) (unit 1)
@@
     (pin "1")
   )
+  (symbol (lib_id "Connector:Conn_01x04_Male") (at 24.638 75.946 0) (unit 1)
+    (in_bom yes) (on_board yes)
+    (property "Reference" "J12" (id 0) (at 25.273 69.63 0))
+    (property "Value" "Conn_01x04_Male" (id 1) (at 27.432 83.058 0))
+    (property "Footprint" "" (id 2) (at 24.638 75.946 0)
+      (effects (font (size 1.27 1.27)) hide)
+    )
+    (property "Datasheet" "~" (id 3) (at 24.638 75.946 0)
+      (effects (font (size 1.27 1.27)) hide)
+    )
+    (pin "1")
+    (pin "2")
+    (pin "3")
+    (pin "4")
+  )
+  (symbol (lib_id "power:GND") (at 32.004 81.026 90) (unit 1)
+    (in_bom yes) (on_board yes) (fields_autoplaced)
+    (property "Reference" "#PWR0123" (id 0) (at 38.354 81.026 0)
+      (effects (font (size 1.27 1.27)) hide)
+    )
+    (property "Value" "GND" (id 1) (at 35.179 81.4598 90)
+      (effects (font (size 1.27 1.27)) (justify right))
+    )
+    (property "Footprint" "" (id 2) (at 32.004 81.026 0)
+      (effects (font (size 1.27 1.27)) hide)
+    )
+    (property "Datasheet" "" (id 3) (at 32.004 81.026 0)
+      (effects (font (size 1.27 1.27)) hide)
+    )
+    (pin "1")
+  )
   (symbol (lib_id "Connector:Conn_01x06_Female") (at 25.908 18.288 90) (unit 1)
     (in_bom yes) (on_board yes)
@@
     (pin "1")
   )
+  (symbol (lib_id "Connector:Conn_01x08_Male") (at 43.434 82.296 0) (unit 1)
+    (in_bom yes) (on_board yes)
+    (property "Reference" "J14" (id 0) (at 44.069 70.9 0))
+    (property "Value" "" (id 1) (at 46.736 94.742 0))
+    (property "Footprint" "" (id 2) (at 43.434 82.296 0)
+      (effects (font (size 1.27 1.27)) hide)
+    )
+    (property "Datasheet" "~" (id 3) (at 43.434 82.296 0)
+      (effects (font (size 1.27 1.27)) hide)
+    )
+    (pin "1")
+    (pin "2")
+    (pin "3")
+    (pin "4")
+    (pin "5")
+    (pin "6")
+    (pin "7")
+    (pin "8")
+  )
   (symbol (lib_id "power:GND") (at 103.632 32.766 0) (unit 1)
     (in_bom yes) (on_board yes) (fields_autoplaced)
@@
     )
     (property "Datasheet" "" (id 3) (at 103.632 32.766 0)
+      (effects (font (size 1.27 1.27)) hide)
+    )
+    (pin "1")
+  )
+  (symbol (lib_id "power:GND") (at 48.514 92.456 90) (unit 1)
+    (in_bom yes) (on_board yes) (fields_autoplaced)
+    (property "Reference" "#PWR0121" (id 0) (at 54.864 92.456 0)
+      (effects (font (size 1.27 1.27)) hide)
+    )
+    (property "Value" "GND" (id 1) (at 51.689 92.8898 90)
+      (effects (font (size 1.27 1.27)) (justify right))
+    )
+    (property "Footprint" "" (id 2) (at 48.514 92.456 0)
+      (effects (font (size 1.27 1.27)) hide)
+    )
+    (property "Datasheet" "" (id 3) (at 48.514 92.456 0)
       (effects (font (size 1.27 1.27)) hide)
     )
@@
     (pin "1")
   )
+  (symbol (lib_id "Connector:Conn_01x04_Male") (at 24.892 90.17 0) (unit 1)
+    (in_bom yes) (on_board yes)
+    (property "Reference" "J13" (id 0) (at 27.94 98.552 0))
+    (property "Value" "Conn_01x04_Male" (id 1) (at 27.94 97.028 0))
+    (property "Footprint" "" (id 2) (at 24.892 90.17 0)
+      (effects (font (size 1.27 1.27)) hide)
+    )
+    (property "Datasheet" "~" (id 3) (at 24.892 90.17 0)
+      (effects (font (size 1.27 1.27)) hide)
+    )
+    (pin "1")
+    (pin "2")
+    (pin "3")
+    (pin "4")
+  )
   (symbol (lib_id "power:GND") (at 41.402 27.178 0) (unit 1)

Commit message: gkg
Parts:
- J1, J2: footprint Connector_PinSocket_2.54mm:PinSocket_1x06_P2.54mm_Vertical -> (none)
Changed lines of the file:
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@@
       (effects (font (size 1.27 1.27)) (justify left))
     )
-    (property "Footprint" "Connector_PinSocket_2.54mm:PinSocket_1x06_P2.54mm_Vertical" (id 2) (at 25.908 18.288 0)
+    (property "Footprint" "" (id 2) (at 25.908 18.288 0)
       (effects (font (size 1.27 1.27)) hide)
     )
@@
       (effects (font (size 1.27 1.27)) (justify left))
     )
-    (property "Footprint" "Connector_PinSocket_2.54mm:PinSocket_1x06_P2.54mm_Vertical" (id 2) (at 46.482 18.288 0)
+    (property "Footprint" "" (id 2) (at 46.482 18.288 0)
       (effects (font (size 1.27 1.27)) hide)
     )

Commit message: 23542
Parts:
- J1, J2: footprint (none) -> Connector_PinHeader_2.54mm:PinHeader_1x06_P2.54mm_Vertical
- J12, J13: footprint (none) -> Connector_PinSocket_2.54mm:PinSocket_1x04_P2.54mm_Vertical
- J14: value (none) -> Conn_01x08_Male; footprint (none) -> Connector_PinSocket_2.54mm:PinSocket_1x08_P2.54mm_Vertical
Changed lines of the file:
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@@
     (property "Reference" "J12" (id 0) (at 25.273 69.63 0))
     (property "Value" "Conn_01x04_Male" (id 1) (at 27.432 83.058 0))
-    (property "Footprint" "" (id 2) (at 24.638 75.946 0)
+    (property "Footprint" "Connector_PinSocket_2.54mm:PinSocket_1x04_P2.54mm_Vertical" (id 2) (at 24.638 75.946 0)
       (effects (font (size 1.27 1.27)) hide)
     )
@@
       (effects (font (size 1.27 1.27)) (justify left))
     )
-    (property "Footprint" "" (id 2) (at 25.908 18.288 0)
+    (property "Footprint" "Connector_PinHeader_2.54mm:PinHeader_1x06_P2.54mm_Vertical" (id 2) (at 25.908 18.288 0)
       (effects (font (size 1.27 1.27)) hide)
     )
@@
     (in_bom yes) (on_board yes)
     (property "Reference" "J14" (id 0) (at 44.069 70.9 0))
-    (property "Value" "" (id 1) (at 46.736 94.742 0))
-    (property "Footprint" "" (id 2) (at 43.434 82.296 0)
+    (property "Value" "Conn_01x08_Male" (id 1) (at 46.736 94.742 0))
+    (property "Footprint" "Connector_PinSocket_2.54mm:PinSocket_1x08_P2.54mm_Vertical" (id 2) (at 43.434 82.296 0)
       (effects (font (size 1.27 1.27)) hide)
     )
@@
       (effects (font (size 1.27 1.27)) (justify left))
     )
-    (property "Footprint" "" (id 2) (at 46.482 18.288 0)
+    (property "Footprint" "Connector_PinHeader_2.54mm:PinHeader_1x06_P2.54mm_Vertical" (id 2) (at 46.482 18.288 0)
       (effects (font (size 1.27 1.27)) hide)
     )
@@
     (property "Reference" "J13" (id 0) (at 27.94 98.552 0))
     (property "Value" "Conn_01x04_Male" (id 1) (at 27.94 97.028 0))
-    (property "Footprint" "" (id 2) (at 24.892 90.17 0)
+    (property "Footprint" "Connector_PinSocket_2.54mm:PinSocket_1x04_P2.54mm_Vertical" (id 2) (at 24.892 90.17 0)
       (effects (font (size 1.27 1.27)) hide)
     )
