File: placas/Laberinto/BluePill/Modularizado/BluePillVersion/BluePillVersion.kicad_pcb (KiCad board)
At the start: 2 copper layers, 20 parts, among them J1 Conn_01x06_Female, J2 Conn_01x06_Female, J3 Conn_01x04_Male, J4 Conn_01x04_Male, J5 Conn_01x04_Male, J6 Conn_01x04_Male, J7 Conn_01x08_Female, J8 Conn_01x02_Male, SW1 SW_Push, SW2 SW_Push, SW3 SW_Push, SW4 SW_DPDT_x2

Commit message: gh
Parts:
- added J10: Conn_01x04_Male, Connector_PinHeader_2.54mm:PinHeader_1x04_P2.54mm_Vertical, B.Cu at (105.9, 42.1)
- added J11: Conn_01x08_Male, Connector_PinHeader_2.54mm:PinHeader_1x08_P2.54mm_Vertical, B.Cu at (14.0, 51.3)
- added J12: Conn_01x04_Male, Connector_PinSocket_2.54mm:PinSocket_1x04_P2.54mm_Vertical, F.Cu at (208.4, 30.2)
- added J13: Conn_01x04_Male, Connector_PinSocket_2.54mm:PinSocket_1x04_P2.54mm_Vertical, F.Cu at (208.4, 41.8)
- added J14: Conn_01x08_Male, Connector_PinSocket_2.54mm:PinSocket_1x08_P2.54mm_Vertical, F.Cu at (115.9, 51.1)
- added J9: Conn_01x04_Male, Connector_PinHeader_2.54mm:PinHeader_1x04_P2.54mm_Vertical, B.Cu at (105.9, 30.3)
- added REF**: SharpHolder, propios:SharpHolder, F.Cu at (68.3, 17.1)
- added REF**: MotorHolder, propios:MotorHolder, F.Cu at (168.9, 74.0)
- added REF**: BolitaHolder, propios:BolitaHolder, F.Cu at (162.2, -6.54)
- added REF**: SharpHolder, propios:SharpHolder, F.Cu at (59.6, 17.2)
- added REF**: SharpHolder, propios:SharpHolder, F.Cu at (30.1, 17.1)
- added REF**: MotorHolder, propios:MotorHolder, F.Cu at (132.7, 74.0)
- added U1: tb6612fng, propios:tb6612fng, F.Cu at (136.8, 19.9)
- added U2: Mt3608, propios:MT3608, F.Cu at (194.8, 22.3)
- added U3: YAAJ_BluePill_Part_Like_SWD_Breakout, Footprints:YAAJ_BluePill_1, F.Cu at (38.6, 50.9)
- J3, J4, J5, R1, R2, R3, R5: moved to B.Cu
- moved D2 220.2 mm to (16.0, 28.1), turned to 180 degrees
- moved SW2 212.5 mm to (25.8, 39.5), turned to 90 degrees
- moved SW1 208.6 mm to (25.8, 49.6), turned to 90 degrees
- moved SW3 200.8 mm to (25.8, 29.6), turned to 90 degrees
- moved J7 193.3 mm to (14.1, 17.4), turned to 90 degrees
- moved R4 188.3 mm to (19.9, 30.6), turned to -90 degrees
- moved R1 178.7 mm to (37.8, 46.6)
- moved J4 178.6 mm to (51.7, 16.5), turned to 180 degrees
- moved J5 177.3 mm to (63.4, 16.5), turned to 90 degrees
- moved J3 172.9 mm to (67.2, 16.5), turned to 180 degrees
- moved R3 170.6 mm to (48.0, 43.1), turned to 180 degrees
- moved R5 169.7 mm to (37.9, 39.5)
- moved J6 155.4 mm to (82.8, 15.6), turned to 90 degrees
- moved J8 153.2 mm to (99.1, 30.3)
- moved D1 147.6 mm to (93.9, 40.8), turned to 180 degrees
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Connections:
- J3 pad 4: /Controlador/SHARP_C -> /Controlador/SHARP_D
- J5 pad 4: /Controlador/SHARP_D -> /Controlador/SHARP_C
Routing:
- net GND: track 0.00 -> 473.9 mm, vias 0 -> 6
- net /Controlador/3.3v: track 0.00 -> 192.0 mm, vias 0 -> 3
- net /Placa Motores/5v: track 0.00 -> 85.5 mm
- net /Controlador/PWMA: track 0.00 -> 85.2 mm, vias 0 -> 2
- net /Placa Motores/VOut: track 0.00 -> 83.1 mm, vias 0 -> 2
- net /Controlador/AIN2: track 0.00 -> 75.1 mm, vias 0 -> 2
- net /Controlador/AIN1: track 0.00 -> 68.5 mm, vias 0 -> 2
- net /Controlador/STBY: track 0.00 -> 67.7 mm
- net /Placa Motores/PWMB: track 0.00 -> 67.0 mm
- net /Controlador/VIn: track 0.00 -> 65.1 mm
- net /Placa Motores/MB2: track 0.00 -> 63.9 mm, vias 0 -> 2
- net /Controlador/BIN1: track 0.00 -> 63.9 mm
- net /Controlador/BIN2: track 0.00 -> 62.6 mm
- net /Placa Motores/MB1: track 0.00 -> 62.1 mm
- net /Placa Motores/BIN2: track 0.00 -> 56.2 mm
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
Commit message: gkg
Parts:
- J1, J2: footprint Connector_PinSocket_2.54mm:PinSocket_1x06_P2.54mm_Vertical -> Connector_PinHeader_2.54mm:PinHeader_1x06_P2.54mm_Vertical
- moved REF** 26.5 mm to (164.2, 19.9)
- moved J1 12.5 mm to (166.8, 54.3)
- moved J2 12.0 mm to (148.5, 54.4)
- moved D2 11.8 mm to (18.0, 39.8)
- moved D3 11.8 mm to (94.6, 44.4)
- moved J14 11.8 mm to (117.9, 62.7)
- moved J4 11.8 mm to (53.7, 28.1)
- moved R5 11.8 mm to (39.9, 51.2)
- moved REF** 11.8 mm to (170.9, 85.6)
- moved SW1 11.8 mm to (27.9, 61.2)
- moved SW2 11.8 mm to (27.9, 51.2)
- moved U3 11.8 mm to (40.6, 62.5)
- moved J10 11.8 mm to (108.0, 53.7)
- moved J11 11.8 mm to (16.0, 62.9)
- moved J12 11.8 mm to (210.5, 41.8)
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Routing:
- net GND: track 473.9 -> 483.6 mm, vias 6 -> 8
- net /Placa Motores/BO2: track 13.8 -> 19.3 mm
- net /Placa Motores/BO1: track 8.78 -> 14.1 mm
- net /Placa Motores/MA2: track 37.6 -> 35.2 mm
- net /Placa Motores/AO2: track 45.8 -> 48.2 mm
- net /Placa Motores/AO1: track 53.7 -> 56.1 mm
- net /Placa Motores/MA1: track 41.8 -> 40.1 mm
- net /Placa Motores/MB2: track 63.9 -> 63.2 mm
- added copper zone on B.Cu, net GND
- added copper zone on F.Cu, net GND

Commit message: sdcdsc
Parts:
- moved J7 17.8 mm to (33.9, 29.2), turned to -90 degrees
Routing:
- net GND: track 483.6 -> 410.5 mm
- net /Controlador/3.3v: track 192.0 -> 138.8 mm, vias 3 -> 1
- net /Controlador/SDA: track 42.5 -> 48.3 mm, vias 0 -> 2
- net /Controlador/STBY: track 67.7 -> 73.0 mm
- net /Controlador/BIN1: track 63.9 -> 67.4 mm
- net /Controlador/BIN2: track 62.6 -> 65.2 mm
- net /Controlador/PWMB: track 53.7 -> 55.9 mm
- net /Controlador/SCL: track 54.4 -> 52.3 mm
- net /Controlador/MA1: track 50.7 -> 52.1 mm
- net /Controlador/MA2: track 46.9 -> 47.8 mm

Commit message: 23542
Parts:
- moved J12 5.08 mm to (205.4, 41.8)
- moved J13 5.08 mm to (205.3, 53.4)
- moved REF** 5.08 mm to (165.8, 85.6)
- moved REF** 5.08 mm to (159.2, 19.9)
- moved REF** 5.08 mm to (129.6, 85.6)
- moved U2 5.08 mm to (191.8, 33.9)
- moved J14 5.08 mm to (112.8, 62.7)
- moved J1 5.08 mm to (161.7, 54.3)
- moved J2 5.08 mm to (143.5, 54.4)
- moved U1 5.08 mm to (133.8, 31.5)
Connections:
- U3 pad 13: /Controlador/MA1 -> unconnected-(U3-Pad13)
- U3 pad 15: /Controlador/PWMA -> /Controlador/MA1
- U3 pad 16: /Controlador/MB1 -> /Controlador/PWMA
- U3 pad 17: /Controlador/MB2 -> /Controlador/PWMB
- U3 pad 5: /Controlador/PWMB -> /Controlador/MB2
- U3 pad 6: unconnected-(U3-Pad6) -> /Controlador/MB1
Routing:
- net /Controlador/3.3v: track 138.8 -> 95.7 mm
- net /Controlador/PWMB: track 55.9 -> 90.0 mm, vias 0 -> 2
- net /Controlador/MB2: track 37.0 -> 67.9 mm, vias 0 -> 2
- net /Controlador/MB1: track 40.9 -> 59.5 mm, vias 0 -> 2
- net /Controlador/PWMA: track 85.2 -> 89.2 mm
- net /Controlador/MA1: track 52.1 -> 48.3 mm, vias 0 -> 2
- net /Controlador/BIN2: track 65.2 -> 68.7 mm
- net /Controlador/STBY: track 73.0 -> 76.3 mm
- net /Controlador/BIN1: track 67.4 -> 70.6 mm

Commit message: dsfdf
Routing:
- net GND: track 410.5 -> 434.7 mm, vias 8 -> 9
- net /Controlador/BTN3: track 31.6 -> 33.1 mm
- net /Controlador/3.3v: track 95.7 -> 94.6 mm
- net /Controlador/BIN1: track 70.6 -> 71.4 mm
- net /Controlador/SCL: track 52.3 -> 51.7 mm
- added copper zone on B.Cu, net /Placa Motores/BIN1
- added copper zone on F.Cu, net /Placa Motores/BIN1

Commit message: 565
Routing:
- removed copper zone on B.Cu, net /Placa Motores/BIN1
- removed copper zone on F.Cu, net /Placa Motores/BIN1
- removed copper zone on B.Cu, net GND
- removed copper zone on F.Cu, net GND

Commit message: 4155456
Parts:
- moved J2 2.64 mm to (146.1, 54.4)
- moved J1 1.42 mm to (163.1, 54.3)
Routing:
- net GND: track 434.7 -> 458.1 mm, vias 9 -> 15
- net /Placa Motores/AO1: track 56.1 -> 62.1 mm
- net /Placa Motores/AO2: track 48.2 -> 54.2 mm
- net /Placa Motores/BO2: track 19.3 -> 14.8 mm
- net /Placa Motores/BO1: track 14.1 -> 9.69 mm
- net /Placa Motores/MB2: track 63.2 -> 60.5 mm
- net /Controlador/Led: track 36.2 -> 38.8 mm, vias 0 -> 1
- net /Placa Motores/5v: track 85.2 -> 87.6 mm
- net /Placa Motores/MA2: track 35.2 -> 33.7 mm
- net /Placa Motores/MA1: track 40.1 -> 38.6 mm
- net /Placa Motores/MB1: track 61.8 -> 60.3 mm
- net /Controlador/MA2: track 47.8 -> 49.1 mm
- net Net-(D2-Pad2): track 10.0 -> 8.87 mm
- net /Controlador/SHARP_C: track 30.7 -> 31.8 mm
- net /Placa Motores/PWMB: track 67.0 -> 65.9 mm
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
Commit message: 23
Parts:
- moved J1 1.42 mm to (161.7, 54.3)
- moved J8 1.32 mm to (101.1, 40.6)
- moved J2 1.07 mm to (145.0, 54.4)
- moved U1 0.26 mm to (134.0, 31.5)
Routing:
- net /Controlador/3.3v: track 94.3 -> 121.9 mm
- net GND: track 458.1 -> 451.2 mm, vias 15 -> 11
- net /Controlador/BTN2: track 21.8 -> 28.3 mm
- net /Controlador/SHARP_D: track 14.4 -> 18.4 mm
- net /Controlador/SHARP_C: track 31.8 -> 34.7 mm
- net /Controlador/Led: track 38.8 -> 36.2 mm, vias 1 -> 0
- net /Placa Motores/AO1: track 62.1 -> 59.7 mm
- net /Placa Motores/VOut: track 84.0 -> 81.6 mm
- net /Placa Motores/AO2: track 54.2 -> 52.1 mm
- net /Placa Motores/MB1: track 60.3 -> 62.4 mm
- net /Placa Motores/BO2: track 14.8 -> 13.4 mm
- net /Placa Motores/BO1: track 9.69 -> 8.28 mm
- net /Controlador/AIN1: track 68.5 -> 69.9 mm
- net Net-(D3-Pad1): track 6.59 -> 7.94 mm
- net /Controlador/5v: track 33.4 -> 34.7 mm
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