File: placas/Laberinto/BluePill/Modularizado/BluePillVersion/BluePillVersion.kicad_pcb (KiCad board)
At the start: 2 copper layers, 35 parts, among them J1 Conn_01x06_Female, J10 Conn_01x04_Male, J11 Conn_01x08_Male, J12 Conn_01x04_Male, J13 Conn_01x04_Male, J14 Conn_01x08_Male, J2 Conn_01x06_Female, J3 Conn_01x04_Male, J4 Conn_01x04_Male, J5 Conn_01x04_Male, J6 Conn_01x04_Male, J7 Conn_01x08_Female, J8 Conn_01x02_Male, J9 Conn_01x04_Male, SW1 SW_Push, SW2 SW_Push, SW3 SW_Push, SW4 SW_DPDT_x2, U1 tb6612fng, U2 Mt3608, U3 YAAJ_BluePill_Part_Like_SWD_B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

Commit message: fdgkl
Connections:
- U3 pad 11: /Controlador/AIN1 -> unconnected-(U3-Pad11)
- U3 pad 13: unconnected-(U3-Pad13) -> /Controlador/AIN1
Routing:
- net /Controlador/AIN1: track 69.9 -> 75.1 mm

Commit message: fg
Parts:
- moved R4 9.96 mm to (21.8, 32.3)
Routing:
- net /Controlador/Led: track 36.2 -> 46.2 mm
- net Net-(D2-Pad2): track 8.86 -> 13.6 mm
- net /Controlador/BIN1: track 71.1 -> 73.0 mm
- net /Controlador/STBY: track 76.0 -> 76.9 mm
Changed lines of the file:
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@@
   )
   (footprint "Resistor_THT:R_Axial_DIN0207_L6.3mm_D2.5mm_P10.16mm_Horizontal" (layer "F.Cu")
-    (at 21.8948 42.2656 -90)
+    (at 21.844 32.3088 -90)
     (descr "Resistor, Axial_DIN0207 series, Axial, Horizontal, pin pitch=10.16mm, 0.25W = 1/4W, length*diameter=6.3*2.5mm^2, http://cdn-reichelt.de/documents/datenblatt/B400/1_4W%23YAG.pdf")
     (tags "Resistor Axial_DIN0207 series Axial Horizontal pin pitch 10.16mm 0.25W = 1/4W length 6.3mm diameter 2.5mm")
@@
   (segment (start 88.646 52.5272) (end 88.646 54.9148) (width 1) (layer "B.Cu") (net 2))
   (segment (start 88.6968 52.4764) (end 88.646 52.5272) (width 1) (layer "B.Cu") (net 2))
-  (segment (start 15.499 42.2198) (end 15.499 39.7764) (width 1) (layer "B.Cu") (net 3))
-  (segment (start 21.8948 42.2656) (end 15.5448 42.2656) (width 1) (layer "B.Cu") (net 3))
-  (segment (start 15.5448 42.2656) (end 15.499 42.2198) (width 1) (layer "B.Cu") (net 3))
+  (segment (start 15.9104 32.3088) (end 21.844 32.3088) (width 1) (layer "B.Cu") (net 3))
+  (segment (start 15.499 39.7764) (end 15.499 32.7202) (width 1) (layer "B.Cu") (net 3))
+  (segment (start 15.499 32.7202) (end 15.9104 32.3088) (width 1) (layer "B.Cu") (net 3))
   (segment (start 101.092 44.45) (end 101.092 43.18) (width 1) (layer "B.Cu") (net 4))
   (segment (start 101.1428 44.5008) (end 101.092 44.45) (width 1) (layer "B.Cu") (net 4))
@@
   (segment (start 53.6956 38.0492) (end 53.7464 37.9984) (width 1) (layer "F.Cu") (net 19))
   (via (at 53.6956 38.0492) (size 2) (drill 1.2) (layers "F.Cu" "B.Cu") (net 19))
-  (segment (start 71.12 44.196) (end 71.12 47.244) (width 1) (layer "B.Cu") (net 19))
-  (segment (start 53.6956 37.9984) (end 53.6956 41.6052) (width 1) (layer "B.Cu") (net 19))
-  (segment (start 69.0372 42.1132) (end 71.12 44.196) (width 1) (layer "B.Cu") (net 19))
-  (segment (start 54.2036 42.1132) (end 69.0372 42.1132) (width 1) (layer "B.Cu") (net 19))
-  (segment (start 53.6956 41.6052) (end 54.2036 42.1132) (width 1) (layer "B.Cu") (net 19))
+  (segment (start 53.6956 37.9984) (end 53.6956 39.4208) (width 1) (layer "B.Cu") (net 19))
+  (segment (start 71.12 42.3672) (end 71.12 47.244) (width 1) (layer "B.Cu") (net 19))
+  (segment (start 56.642 42.3672) (end 71.12 42.3672) (width 1) (layer "B.Cu") (net 19))
+  (segment (start 53.6956 39.4208) (end 56.642 42.3672) (width 1) (layer "B.Cu") (net 19))
   (segment (start 76.0984 47.1424) (end 76.2 47.244) (width 1) (layer "B.Cu") (net 21))
   (segment (start 69.2404 35.7632) (end 75.8952 35.7632) (width 1) (layer "B.Cu") (net 21))
@@
   (segment (start 36.4236 58.4708) (end 25.2476 58.4708) (width 1) (layer "F.Cu") (net 33))
   (segment (start 48.26 62.484) (end 48.26 60.3504) (width 1) (layer "F.Cu") (net 33))
+  (segment (start 21.8948 55.118) (end 21.844 55.0672) (width 1) (layer "F.Cu") (net 33))
+  (segment (start 21.844 55.0672) (end 21.844 42.4688) (width 1) (layer "F.Cu") (net 33))
   (segment (start 36.4236 60.0456) (end 36.4236 58.4708) (width 1) (layer "F.Cu") (net 33))
   (segment (start 47.9552 60.0456) (end 36.4236 60.0456) (width 1) (layer "F.Cu") (net 33))
   (segment (start 25.2476 58.4708) (end 25.2476 55.118) (width 1) (layer "F.Cu") (net 33))
   (segment (start 25.2476 55.118) (end 21.8948 55.118) (width 1) (layer "F.Cu") (net 33))
-  (segment (start 21.8948 55.118) (end 21.8948 52.4256) (width 1) (layer "F.Cu") (net 33))
   (segment (start 45.6692 51.2064) (end 37.6936 51.2064) (width 1) (layer "B.Cu") (net 34))
   (segment (start 45.72 62.484) (end 45.72 51.1556) (width 1) (layer "B.Cu") (net 34))
@@
   (segment (start 58.42 69.596) (end 24.384 69.596) (width 1) (layer "B.Cu") (net 42))
   (segment (start 17.8308 50.2412) (end 17.8158 50.2262) (width 1) (layer "B.Cu") (net 42))
-  (segment (start 19.2382 52.7662) (end 22.606 56.134) (width 1) (layer "B.Cu") (net 43))
-  (segment (start 16.002 52.7662) (end 19.2382 52.7662) (width 1) (layer "B.Cu") (net 43))
   (segment (start 60.96 71.6788) (end 60.96 62.484) (width 1) (layer "B.Cu") (net 43))
   (segment (start 22.606 71.6788) (end 60.96 71.6788) (width 1) (layer "B.Cu") (net 43))
-  (segment (start 22.606 56.134) (end 22.606 71.6788) (width 1) (layer "B.Cu") (net 43))
-  (segment (start 21.082 56.896) (end 19.4922 55.3062) (width 1) (layer "B.Cu") (net 44))
-  (segment (start 19.4922 55.3062) (end 16.002 55.3062) (width 1) (layer "B.Cu") (net 44))
-  (segment (start 21.082 73.6092) (end 21.082 56.896) (width 1) (layer "B.Cu") (net 44))
+  (segment (start 22.5402 52.7662) (end 22.606 52.832) (width 1) (layer "B.Cu") (net 43))
+  (segment (start 16.002 52.7662) (end 22.5402 52.7662) (width 1) (layer "B.Cu") (net 43))
+  (segment (start 22.606 52.832) (end 22.606 71.6788) (width 1) (layer "B.Cu") (net 43))
+  (segment (start 63.5 73.6092) (end 21.082 73.6092) (width 1) (layer "B.Cu") (net 44))
+  (segment (start 21.082 73.6092) (end 21.082 55.3062) (width 1) (layer "B.Cu") (net 44))
+  (segment (start 21.082 55.3062) (end 16.002 55.3062) (width 1) (layer "B.Cu") (net 44))
   (segment (start 63.5 62.484) (end 63.5 73.6092) (width 1) (layer "B.Cu") (net 44))
-  (segment (start 63.5 73.6092) (end 21.082 73.6092) (width 1) (layer "B.Cu") (net 44))
   (segment (start 22.9108 70.104) (end 22.9108 57.9628) (width 1) (layer "F.Cu") (net 45))
   (segment (start 22.9108 57.9628) (end 22.7584 57.8104) (width 1) (layer "F.Cu") (net 45))
