File: placas/Laberinto/BluePill/Modularizado/BluePillVersion V2/BluePillVersion.kicad_pcb (KiCad board)
At the start: 2 copper layers, 95.3 x 95.2 mm, 29 parts, among them J1 Conn_01x06_Female, J2 Conn_01x06_Female, J3 Conn_01x04_Male, J4 Conn_01x04_Male, J5 Conn_01x04_Male, J6 Conn_01x04_Male, J7 Conn_01x04_Female, J8 Conn_01x08_Female, J9 Conn_01x02_Male, SW1 SW_Push, SW2 SW_Push, SW3 SW_Push, SW4 SW_DPDT_x2, U1 tb6612fng, U2 YAAJ_BluePill_Part_Like_SWD_B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, U3 Mt3608, U4 Mini360

Commit message: gdfgfg
Routing:
- net /MA1: track 152.7 -> 158.2 mm
- net /3.3v: track 275.1 -> 274.6 mm

Commit message: ffb
Routing:
- net /PWMA: track 29.6 -> 30.2 mm
Changed lines of the file:
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@@
   (segment (start 201.0664 31.8516) (end 201.0664 29.972) (width 1) (layer "B.Cu") (net 19))
   (segment (start 189.2658 102.4486) (end 181.6608 94.8436) (width 1) (layer "B.Cu") (net 19))
-  (segment (start 251.01038 40.42922) (end 211.21882 40.42922) (width 1) (layer "B.Cu") (net 19))
   (segment (start 201.0664 29.972) (end 200.2536 29.1592) (width 1) (layer "B.Cu") (net 19))
   (segment (start 200.2536 29.1592) (end 195.3768 29.1592) (width 1) (layer "B.Cu") (net 19))
   (segment (start 227.6184 59.8424) (end 227.6156 59.8396) (width 1) (layer "B.Cu") (net 19))
+  (segment (start 258.3588 35.2044) (end 258.3588 37.7952) (width 1) (layer "B.Cu") (net 19))
   (segment (start 244.1956 50.546) (end 242.2652 50.546) (width 1) (layer "B.Cu") (net 19))
   (segment (start 205.8924 35.1028) (end 206.1464 35.3568) (width 1) (layer "B.Cu") (net 19))
   (segment (start 206.1464 35.3568) (end 206.1464 37.2872) (width 1) (layer "B.Cu") (net 19))
-  (segment (start 258.3588 37.7952) (end 253.6444 37.7952) (width 1) (layer "B.Cu") (net 19))
   (segment (start 240.3856 59.8424) (end 227.6184 59.8424) (width 1) (layer "B.Cu") (net 19))
   (segment (start 180.594 43.7388) (end 176.3776 43.7388) (width 1) (layer "B.Cu") (net 19))
@@
   (segment (start 250.444 50.55928) (end 244.25968 50.55928) (width 1) (layer "B.Cu") (net 19))
   (segment (start 195.2244 25.4508) (end 195.2244 22.6568) (width 1) (layer "B.Cu") (net 19))
+  (segment (start 253.6444 37.7952) (end 251.01038 40.42922) (width 1) (layer "B.Cu") (net 19))
   (segment (start 240.6396 59.5884) (end 240.3856 59.8424) (width 1) (layer "B.Cu") (net 19))
   (segment (start 195.3768 29.1592) (end 195.2244 29.0068) (width 1) (layer "B.Cu") (net 19))
   (segment (start 176.3776 43.7388) (end 175.3616 42.7228) (width 1) (layer "B.Cu") (net 19))
+  (segment (start 258.3588 37.7952) (end 253.6444 37.7952) (width 1) (layer "B.Cu") (net 19))
   (segment (start 201.168 35.1028) (end 205.8924 35.1028) (width 1) (layer "B.Cu") (net 19))
+  (segment (start 216.90842 40.42922) (end 211.836 35.3568) (width 1) (layer "B.Cu") (net 19))
   (segment (start 244.25968 50.55928) (end 244.2464 50.546) (width 1) (layer "B.Cu") (net 19))
   (segment (start 175.3616 19.05) (end 175.5648 18.8468) (width 1) (layer "B.Cu") (net 19))
@@
   (segment (start 195.2244 29.0068) (end 195.2244 25.4508) (width 1) (layer "B.Cu") (net 19))
   (segment (start 201.0664 31.8516) (end 201.0664 35.0012) (width 1) (layer "B.Cu") (net 19))
-  (segment (start 211.21882 40.42922) (end 206.1464 35.3568) (width 1) (layer "B.Cu") (net 19))
-  (segment (start 258.3588 35.2044) (end 258.3588 37.7952) (width 1) (layer "B.Cu") (net 19))
+  (segment (start 211.836 35.3568) (end 206.1464 35.3568) (width 1) (layer "B.Cu") (net 19))
   (segment (start 206.1464 43.688) (end 206.1464 37.2872) (width 1) (layer "B.Cu") (net 19))
+  (segment (start 251.01038 40.42922) (end 216.90842 40.42922) (width 1) (layer "B.Cu") (net 19))
   (segment (start 175.5648 18.8468) (end 195.2244 18.8468) (width 1) (layer "B.Cu") (net 19))
-  (segment (start 253.6444 37.7952) (end 251.01038 40.42922) (width 1) (layer "B.Cu") (net 19))
   (segment (start 181.6608 56.3372) (end 180.594 55.2704) (width 1) (layer "B.Cu") (net 19))
   (segment (start 180.594 55.2704) (end 180.594 43.7388) (width 1) (layer "B.Cu") (net 19))
@@
   (segment (start 188.6204 29.6672) (end 188.67 29.7168) (width 1) (layer "B.Cu") (net 30))
   (segment (start 195.9864 37.2872) (end 201.0156 37.2872) (width 1) (layer "B.Cu") (net 30))
-  (segment (start 233.0196 54.356) (end 215.9 54.356) (width 1) (layer "F.Cu") (net 31))
-  (segment (start 234.0864 53.2892) (end 233.0196 54.356) (width 1) (layer "F.Cu") (net 31))
-  (via (at 234.0864 53.2892) (size 2) (drill 1.2) (layers "F.Cu" "B.Cu") (net 31))
+  (segment (start 234.0864 54.356) (end 215.9 54.356) (width 1) (layer "F.Cu") (net 31))
+  (segment (start 234.0864 52.6288) (end 234.0864 54.356) (width 1) (layer "F.Cu") (net 31))
+  (via (at 234.0864 52.6288) (size 2) (drill 1.2) (layers "F.Cu" "B.Cu") (net 31))
   (via (at 215.9 54.356) (size 2) (drill 1.2) (layers "F.Cu" "B.Cu") (net 31))
   (segment (start 212.3756 57.2996) (end 212.9564 57.2996) (width 1) (layer "B.Cu") (net 31))
-  (segment (start 234.0864 53.2892) (end 234.0864 47.0916) (width 1) (layer "B.Cu") (net 31))
+  (segment (start 234.0864 52.6288) (end 234.0864 47.0916) (width 1) (layer "B.Cu") (net 31))
   (segment (start 212.9564 57.2996) (end 215.9 54.356) (width 1) (layer "B.Cu") (net 31))
   (segment (start 223.9264 47.0916) (end 223.9264 51.2064) (width 1) (layer "B.Cu") (net 32))
@@
   (segment (start 211.0232 49.4284) (end 216.2048 49.4284) (width 1) (layer "B.Cu") (net 36))
   (segment (start 216.3064 49.3268) (end 216.3064 47.0916) (width 1) (layer "B.Cu") (net 36))
-  (segment (start 236.6264 54.4576) (end 235.712 55.372) (width 1) (layer "B.Cu") (net 37))
-  (segment (start 225.6536 55.372) (end 215.4428 65.5828) (width 1) (layer "B.Cu") (net 37))
   (segment (start 215.4428 65.5828) (end 215.4428 72.486) (width 1) (layer "B.Cu") (net 37))
-  (segment (start 235.712 55.372) (end 225.6536 55.372) (width 1) (layer "B.Cu") (net 37))
-  (segment (start 215.4428 72.486) (end 215.3892 72.5396) (width 1) (layer "B.Cu") (net 37))
+  (segment (start 236.3724 54.7116) (end 226.314 54.7116) (width 1) (layer "B.Cu") (net 37))
+  (segment (start 226.314 54.7116) (end 215.4428 65.5828) (width 1) (layer "B.Cu") (net 37))
   (segment (start 215.3892 72.5396) (end 212.3756 72.5396) (width 1) (layer "B.Cu") (net 37))
   (segment (start 236.6264 47.0916) (end 236.6264 54.4576) (width 1) (layer "B.Cu") (net 37))
+  (segment (start 215.4428 72.486) (end 215.3892 72.5396) (width 1) (layer "B.Cu") (net 37))
+  (segment (start 236.6264 54.4576) (end 236.3724 54.7116) (width 1) (layer "B.Cu") (net 37))
   (segment (start 247.5972 95.1464) (end 246.38 96.3636) (width 1) (layer "B.Cu") (net 38))
   (segment (start 246.4308 96.4144) (end 246.4308 99.4664) (width 1) (layer "B.Cu") (net 38))
