File: placas/Sumo/Motores/SMD DOBLE/SMD DOBLE/SMD DOBLE.kicad_pcb (KiCad board)
At the start: 2 copper layers, 8 parts, among them J1 Conn_02x04_Odd_Even, J2 Conn_01x02_Male, J3 Conn_01x02_Male, J4 Conn_01x02_Male, U1 VNH2SP30, U2 VNH2SP30

Commit message: fgdgf
Routing:
- net /VCCM: track 172.6 -> 173.5 mm
Changed lines of the file:
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@@
   (via (at 17.526 33.274) (size 1.8) (drill 1) (layers "F.Cu" "B.Cu") (net 1))
   (via (at 17.9832 61.4172) (size 1.8) (drill 1) (layers "F.Cu" "B.Cu") (net 1))
-  (segment (start 9.144 31.305378) (end 12.102978 28.3464) (width 0.5) (layer "B.Cu") (net 1))
   (segment (start 13.6144 37.1856) (end 17.526 33.274) (width 1.2) (layer "B.Cu") (net 1))
-  (segment (start 9.144 35.4076) (end 9.144 31.305378) (width 0.5) (layer "B.Cu") (net 1))
+  (segment (start 12.2428 37.1856) (end 10.922 37.1856) (width 0.5) (layer "B.Cu") (net 1))
   (segment (start 12.2428 37.1856) (end 13.6144 37.1856) (width 1.2) (layer "B.Cu") (net 1))
+  (segment (start 17.526 33.274) (end 17.526 33.8836) (width 0.5) (layer "B.Cu") (net 1))
+  (segment (start 10.922 37.1856) (end 9.144 35.4076) (width 0.5) (layer "B.Cu") (net 1))
+  (segment (start 9.144 29.6672) (end 10.4648 28.3464) (width 0.5) (layer "B.Cu") (net 1))
+  (segment (start 9.144 35.4076) (end 9.144 29.6672) (width 0.5) (layer "B.Cu") (net 1))
   (segment (start 46.7868 28.3464) (end 47.1424 28.702) (width 0.5) (layer "B.Cu") (net 1))
-  (segment (start 10.922 37.1856) (end 9.144 35.4076) (width 0.5) (layer "B.Cu") (net 1))
-  (segment (start 12.2428 37.1856) (end 10.922 37.1856) (width 0.5) (layer "B.Cu") (net 1))
-  (segment (start 17.526 33.274) (end 17.526 33.8836) (width 0.5) (layer "B.Cu") (net 1))
-  (segment (start 12.102978 28.3464) (end 46.7868 28.3464) (width 0.5) (layer "B.Cu") (net 1))
+  (segment (start 10.4648 28.3464) (end 46.7868 28.3464) (width 0.5) (layer "B.Cu") (net 1))
   (segment (start 40.7924 59.182) (end 40.7924 53.3908) (width 0.5) (layer "F.Cu") (net 2))
   (segment (start 40.5892 40.8432) (end 40.5892 35.56) (width 0.5) (layer "F.Cu") (net 2))
@@
         (xy 42.4688 52.2732)
         (xy 42.4688 56.134)
-        (xy 29.3116 56.134)
-        (xy 29.3116 47.6504)
+        (xy 29.4132 56.134)
+        (xy 29.4132 47.6504)
         (xy 49.2252 47.6504)
       )
@@
     (polygon
       (pts
-        (xy 28.9052 66.2432)
+        (xy 28.6512 66.2432)
         (xy 15.9512 66.2432)
         (xy 15.9512 39.6748)
@@
         (xy 19.558 31.6992)
         (xy 19.558 29.0068)
-        (xy 28.9052 29.0068)
-      )
-    )
+        (xy 28.6512 29.0068)
+      )
+    )
