File: placas/Sumo/Motores/SMD DOBLE/SMD DOBLE/SMD DOBLE.kicad_sch (KiCad schematic)
At the start: 8 parts, among them J2 Conn_01x02_Male, J3 Conn_01x02_Male, J4 Conn_01x02_Male, U1 VNH2SP30, U2 VNH2SP30

Commit message: fgdgf
Parts:
- J1: value (none) -> Conn_02x04_Odd_Even; footprint (none) -> Connector_IDC:IDC-Header_2x04_P2.54mm_Vertical
Changed lines of the file:
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@@
     (in_bom yes) (on_board yes) (fields_autoplaced)
     (property "Reference" "J1" (id 0) (at 92.202 15.8582 0))
-    (property "Value" "" (id 1) (at 92.202 18.3951 0))
-    (property "Footprint" "" (id 2) (at 90.932 23.368 0)
+    (property "Value" "Conn_02x04_Odd_Even" (id 1) (at 92.202 18.3951 0))
+    (property "Footprint" "Connector_IDC:IDC-Header_2x04_P2.54mm_Vertical" (id 2) (at 90.932 23.368 0)
       (effects (font (size 1.27 1.27)) hide)
     )
