File: placas/Sumo/placa centra/THT/THT.kicad_pcb (KiCad board)
At the start: 2 copper layers, 57.8 x 47.3 mm, 7 parts, among them J1 Control Piso, J2 BATERIA, J3 Control Motores, J4 Control Sensores, J5 Control Botones, U1 YAAJ_BluePill_Part_Like_SWD_B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

Commit message: yho
Connections:
- net /48Kh renamed /38Kh
Other:
- board size 57.8 x 47.3 mm -> 60.2 x 49.9 mm
Changed lines of the file:
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@@
   (net 33 "unconnected-(U1-Pad21)")
   (net 34 "unconnected-(U1-Pad20)")
-  (net 35 "/48Kh")
-  (net 36 "/B1")
-  (net 37 "/L1")
-  (net 38 "/E2")
-  (net 39 "/E1")
-  (net 40 "/5v")
-  (net 41 "unconnected-(J4-Pad6)")
+  (net 35 "/B1")
+  (net 36 "/L1")
+  (net 37 "/E2")
+  (net 38 "/E1")
+  (net 39 "/5v")
+  (net 40 "unconnected-(J4-Pad6)")
+  (net 41 "/38Kh")
   (footprint "Connector_PinHeader_2.54mm:PinHeader_1x04_P2.54mm_Horizontal" (layer "F.Cu")
     (at 94.6404 76.1492 -90)
@@
       (net 1 "/GND") (pinfunction "Pin_1") (pintype "passive"))
     (pad "2" thru_hole circle (at 5.08 0) (size 3 3) (drill 1.52) (layers *.Cu *.Mask)
-      (net 39 "/E1") (pinfunction "Pin_2") (pintype "passive"))
+      (net 38 "/E1") (pinfunction "Pin_2") (pintype "passive"))
     (model "${KICAD6_3DMODEL_DIR}/TerminalBlock.3dshapes/TerminalBlock_bornier-2_P5.08mm.wrl"
       (offset (xyz 2.539999962 0 0))
@@
       (net 18 "/S5") (pinfunction "PB15") (pintype "bidirectional"))
     (pad "5" thru_hole circle (at 0 10.16 270) (size 1.7 1.7) (drill 1) (layers *.Cu *.Mask)
-      (net 35 "/48Kh") (pinfunction "PA8") (pintype "bidirectional"))
+      (net 41 "/38Kh") (pinfunction "PA8") (pintype "bidirectional"))
     (pad "6" thru_hole circle (at 0 12.7 270) (size 1.7 1.7) (drill 1) (layers *.Cu *.Mask)
       (net 16 "/S1") (pinfunction "PA9") (pintype "bidirectional"))
@@
       (net 22 "/B2") (pinfunction "PB4") (pintype "bidirectional"))
     (pad "13" thru_hole circle (at 0 30.48 270) (size 1.7 1.7) (drill 1) (layers *.Cu *.Mask)
-      (net 36 "/B1") (pinfunction "PB5") (pintype "bidirectional"))
+      (net 35 "/B1") (pinfunction "PB5") (pintype "bidirectional"))
     (pad "14" thru_hole circle (at 0 33.02 270) (size 1.7 1.7) (drill 1) (layers *.Cu *.Mask)
-      (net 37 "/L1") (pinfunction "PB6") (pintype "bidirectional"))
+      (net 36 "/L1") (pinfunction "PB6") (pintype "bidirectional"))
     (pad "15" thru_hole circle (at 0 35.56 270) (size 1.7 1.7) (drill 1) (layers *.Cu *.Mask)
       (net 23 "/L2") (pinfunction "PB7") (pintype "bidirectional"))
@@
       (net 27 "/L4") (pinfunction "PB9") (pintype "bidirectional"))
     (pad "18" thru_hole circle (at 0 43.18 270) (size 1.7 1.7) (drill 1) (layers *.Cu *.Mask)
-      (net 40 "/5v") (pinfunction "5V") (pintype "power_in"))
+      (net 39 "/5v") (pinfunction "5V") (pintype "power_in"))
     (pad "19" thru_hole circle (at 0 45.72 270) (size 1.7 1.7) (drill 1) (layers *.Cu *.Mask)
       (net 1 "/GND") (pinfunction "GND") (pintype "power_in"))
@@
     (fp_line (start 3.135 -1.85) (end 3.135 1.85) (layer "F.Fab") (width 0.1))
     (pad "1" thru_hole rect (at 0 0) (size 2.8 2.8) (drill 1.4) (layers *.Cu *.Mask)
-      (net 38 "/E2") (pinfunction "A") (pintype "passive"))
+      (net 37 "/E2") (pinfunction "A") (pintype "passive"))
     (pad "2" thru_hole oval (at 12.7 0) (size 2.8 2.8) (drill 1.4) (layers *.Cu *.Mask)
-      (net 40 "/5v") (pinfunction "K") (pintype "passive"))
+      (net 39 "/5v") (pinfunction "K") (pintype "passive"))
     (model "${KICAD6_3DMODEL_DIR}/Diode_THT.3dshapes/D_5W_P12.70mm_Horizontal.wrl"
       (offset (xyz 0 0 0))
@@
     (fp_line (start -3.18 15.26) (end -3.18 -4.1) (layer "F.Fab") (width 0.1))
     (pad "1" thru_hole roundrect (at 0 0 270) (size 1.7 1.7) (drill 1) (layers *.Cu *.Mask) (roundrect_rratio 0.147059)
-      (net 36 "/B1") (pinfunction "Pin_1") (pintype "passive"))
+      (net 35 "/B1") (pinfunction "Pin_1") (pintype "passive"))
     (pad "2" thru_hole circle (at 2.54 0 270) (size 1.7 1.7) (drill 1) (layers *.Cu *.Mask)
-      (net 37 "/L1") (pinfunction "Pin_2") (pintype "passive"))
+      (net 36 "/L1") (pinfunction "Pin_2") (pintype "passive"))
     (pad "3" thru_hole circle (at 0 2.54 270) (size 1.7 1.7) (drill 1) (layers *.Cu *.Mask)
       (net 22 "/B2") (pinfunction "Pin_3") (pintype "passive"))
@@
       (net 27 "/L4") (pinfunction "Pin_8") (pintype "passive"))
     (pad "9" thru_hole circle (at 0 10.16 270) (size 1.7 1.7) (drill 1) (layers *.Cu *.Mask)
-      (net 39 "/E1") (pinfunction "Pin_9") (pintype "passive"))
+      (net 38 "/E1") (pinfunction "Pin_9") (pintype "passive"))
     (pad "10" thru_hole circle (at 2.54 10.16 270) (size 1.7 1.7) (drill 1) (layers *.Cu *.Mask)
-      (net 38 "/E2") (pinfunction "Pin_10") (pintype "passive"))
+      (net 37 "/E2") (pinfunction "Pin_10") (pintype "passive"))
     (model "${KICAD6_3DMODEL_DIR}/Connector_IDC.3dshapes/IDC-Header_2x05_P2.54mm_Vertical.wrl"
       (offset (xyz 0 0 0))
@@
       (net 17 "/S4") (pinfunction "Pin_4") (pintype "passive"))
     (pad "5" thru_hole circle (at 0 5.08 90) (size 1.7 1.7) (drill 1) (layers *.Cu *.Mask)
-      (net 35 "/48Kh") (pinfunction "Pin_5") (pintype "passive"))
+      (net 41 "/38Kh") (pinfunction "Pin_5") (pintype "passive"))
     (pad "6" thru_hole circle (at 2.54 5.08 90) (size 1.7 1.7) (drill 1) (layers *.Cu *.Mask)
-      (net 41 "unconnected-(J4-Pad6)") (pinfunction "Pin_6") (pintype "passive+no_connect"))
+      (net 40 "unconnected-(J4-Pad6)") (pinfunction "Pin_6") (pintype "passive+no_connect"))
     (pad "7" thru_hole circle (at 0 7.62 90) (size 1.7 1.7) (drill 1) (layers *.Cu *.Mask)
       (net 18 "/S5") (pinfunction "Pin_7") (pintype "passive"))
@@
     )
   )
-  (gr_rect (start 125.984 84.3788) (end 68.2244 37.084) (layer "Edge.Cuts") (width 0.2) (fill none))
+  (gr_rect (start 127.4572 85.852) (end 67.2592 35.9156) (layer "Edge.Cuts") (width 0.2) (fill none))
   (gr_text "-   +" (at 75.946 83.2104) (layer "F.SilkS")
     (effects (font (size 1.5 1.5) (thickness 0.3)))
@@
   (segment (start 81.8896 52.9844) (end 81.8896 45.5168) (width 1) (layer "B.Cu") (net 27))
   (segment (start 81.8896 45.5168) (end 82.042 45.3644) (width 1) (layer "B.Cu") (net 27))
-  (segment (start 112.3696 52.9844) (end 112.3696 45.2533) (width 1) (layer "B.Cu") (net 35))
-  (segment (start 92.0496 52.9844) (end 92.0496 42.8244) (width 1) (layer "B.Cu") (net 36))
-  (segment (start 92.0496 42.8244) (end 89.662 42.8244) (width 1) (layer "B.Cu") (net 36))
-  (segment (start 89.5096 52.9844) (end 89.5096 45.5168) (width 1) (layer "B.Cu") (net 37))
-  (segment (start 89.5096 45.5168) (end 89.662 45.3644) (width 1) (layer "B.Cu") (net 37))
-  (segment (start 71.1708 46.6344) (end 71.1708 58.8264) (width 1) (layer "B.Cu") (net 38))
-  (segment (start 72.4408 45.3644) (end 71.1708 46.6344) (width 1) (layer "B.Cu") (net 38))
-  (segment (start 72.4408 45.3644) (end 79.502 45.3644) (width 1) (layer "B.Cu") (net 38))
-  (segment (start 72.3392 59.9948) (end 74.9808 59.9948) (width 1) (layer "B.Cu") (net 38))
-  (segment (start 71.1708 58.8264) (end 72.3392 59.9948) (width 1) (layer "B.Cu") (net 38))
-  (segment (start 69.2404 43.18) (end 69.596 42.8244) (width 1) (layer "B.Cu") (net 39))
-  (segment (start 77.724 82.4992) (end 70.7136 82.4992) (width 1) (layer "B.Cu") (net 39))
-  (segment (start 70.7136 82.4992) (end 69.2404 81.026) (width 1) (layer "B.Cu") (net 39))
-  (segment (start 79.502 42.8244) (end 69.596 42.8244) (width 1) (layer "B.Cu") (net 39))
-  (segment (start 78.5876 81.6356) (end 77.724 82.4992) (width 1) (layer "B.Cu") (net 39))
-  (segment (start 78.5876 78.3844) (end 78.5876 81.6356) (width 1) (layer "B.Cu") (net 39))
-  (segment (start 69.2404 81.026) (end 69.2404 43.18) (width 1) (layer "B.Cu") (net 39))
-  (segment (start 84.582 59.9948) (end 79.3496 54.7624) (width 1) (layer "B.Cu") (net 40))
-  (segment (start 87.6808 59.9948) (end 84.582 59.9948) (width 1) (layer "B.Cu") (net 40))
-  (segment (start 79.3496 54.7624) (end 79.3496 52.9844) (width 1) (layer "B.Cu") (net 40))
+  (segment (start 92.0496 52.9844) (end 92.0496 42.8244) (width 1) (layer "B.Cu") (net 35))
+  (segment (start 92.0496 42.8244) (end 89.662 42.8244) (width 1) (layer "B.Cu") (net 35))
+  (segment (start 89.5096 52.9844) (end 89.5096 45.5168) (width 1) (layer "B.Cu") (net 36))
+  (segment (start 89.5096 45.5168) (end 89.662 45.3644) (width 1) (layer "B.Cu") (net 36))
+  (segment (start 71.1708 46.6344) (end 71.1708 58.8264) (width 1) (layer "B.Cu") (net 37))
+  (segment (start 72.4408 45.3644) (end 71.1708 46.6344) (width 1) (layer "B.Cu") (net 37))
+  (segment (start 72.4408 45.3644) (end 79.502 45.3644) (width 1) (layer "B.Cu") (net 37))
+  (segment (start 72.3392 59.9948) (end 74.9808 59.9948) (width 1) (layer "B.Cu") (net 37))
+  (segment (start 71.1708 58.8264) (end 72.3392 59.9948) (width 1) (layer "B.Cu") (net 37))
+  (segment (start 69.2404 43.18) (end 69.596 42.8244) (width 1) (layer "B.Cu") (net 38))
+  (segment (start 77.724 82.4992) (end 70.7136 82.4992) (width 1) (layer "B.Cu") (net 38))
+  (segment (start 70.7136 82.4992) (end 69.2404 81.026) (width 1) (layer "B.Cu") (net 38))
+  (segment (start 79.502 42.8244) (end 69.596 42.8244) (width 1) (layer "B.Cu") (net 38))
+  (segment (start 78.5876 81.6356) (end 77.724 82.4992) (width 1) (layer "B.Cu") (net 38))
+  (segment (start 78.5876 78.3844) (end 78.5876 81.6356) (width 1) (layer "B.Cu") (net 38))
+  (segment (start 69.2404 81.026) (end 69.2404 43.18) (width 1) (layer "B.Cu") (net 38))
+  (segment (start 84.582 59.9948) (end 79.3496 54.7624) (width 1) (layer "B.Cu") (net 39))
+  (segment (start 87.6808 59.9948) (end 84.582 59.9948) (width 1) (layer "B.Cu") (net 39))
+  (segment (start 79.3496 54.7624) (end 79.3496 52.9844) (width 1) (layer "B.Cu") (net 39))
+  (segment (start 112.3696 52.9844) (end 112.3696 45.2533) (width 1) (layer "B.Cu") (net 41))
 )
