File: placas/Sumo/placa centra/THT/THT.kicad_sch (KiCad schematic)
At the start: 7 parts, among them J1 Control Piso, J2 BATERIA, J3 Control Motores, U1 YAAJ_BluePill_Part_Like_SWD_B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

Commit message: fsdf
Parts:
- J4: value (none) -> Control Sensores; footprint (none) -> Connector_IDC:IDC-Header_2x05_P2.54mm_Vertical
- J5: value (none) -> Control Botones
Changed lines of the file:
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@@
     (in_bom yes) (on_board yes) (fields_autoplaced)
     (property "Reference" "J5" (id 0) (at 81.534 53.1962 0))
-    (property "Value" "" (id 1) (at 81.534 55.7331 0))
+    (property "Value" "Control Botones" (id 1) (at 81.534 55.7331 0))
     (property "Footprint" "Connector_IDC:IDC-Header_2x05_P2.54mm_Vertical" (id 2) (at 80.264 63.246 0)
       (effects (font (size 1.27 1.27)) hide)
@@
     (in_bom yes) (on_board yes)
     (property "Reference" "J4" (id 0) (at 64.516 38.2102 0))
-    (property "Value" "" (id 1) (at 64.77 39.878 0))
-    (property "Footprint" "" (id 2) (at 63.246 48.26 0)
+    (property "Value" "Control Sensores" (id 1) (at 64.77 39.878 0))
+    (property "Footprint" "Connector_IDC:IDC-Header_2x05_P2.54mm_Vertical" (id 2) (at 63.246 48.26 0)
       (effects (font (size 1.27 1.27)) hide)
     )
