File: placas/Sumo/alimentacion/THT/THT.kicad_sch (KiCad schematic)
At the start: 6 parts

Commit message: fgdgf
Parts:
- added D1: LED, LED_THT:LED_D3.0mm, symbol Device:LED
- added D2: DIODE, Diode_THT:D_5W_P12.70mm_Horizontal, symbol Simulation_SPICE:DIODE
- added J5: (no value), symbol Connector:Screw_Terminal_01x02
- added R1: R, Resistor_THT:R_Axial_DIN0207_L6.3mm_D2.5mm_P10.16mm_Horizontal, symbol Device:R
- added SW1: (no value), symbol Switch:SW_DPDT_x2
- J1, J2, J3, J4, J6: renamed from J?; value Screw_Terminal_01x02 -> (none)
- gave numbers to parts that had none: 1
Connections:
- net 5v: now also J3.2 (Pin_2), J4.2 (Pin_2), J5.2 (Pin_2)
- net GND: now also J1.1 (Pin_1), J2.1 (Pin_1), J3.1 (Pin_1), J4.1 (Pin_1), D1.1 (K), J5.1 (Pin_1)
- net VCC: now also J1.2 (Pin_2), J2.2 (Pin_2), D2.1 (A); no longer U1.2 (IN+)
- new net: D2.2 (K), SW1.2 (B)
- new net: D1.2 (A), R1.1
- new net VIN: R1.2, SW1.1 (A), U1.2 (IN+)
- no-connect marks 0 -> 1
Other:
- moved on the sheet: J1, J2, J3, J4, J6, U1

Commit message: wed
Parts:
- J1: value (none) -> SENSORES; footprint (none) -> TerminalBlock:TerminalBlock_bornier-2_P5.08mm
- J2: value (none) -> MOTORES; footprint (none) -> Connector_AMASS:AMASS_XT30U-F_1x02_P5.0mm_Vertical
- J3: value (none) -> BOTONES; footprint (none) -> TerminalBlock:TerminalBlock_bornier-2_P5.08mm
- J4: value (none) -> CENTRAL; footprint (none) -> TerminalBlock:TerminalBlock_bornier-2_P5.08mm
- J5: value (none) -> PISO; footprint (none) -> TerminalBlock:TerminalBlock_bornier-2_P5.08mm
- J6: value (none) -> BATERIA; footprint (none) -> Connector_AMASS:AMASS_XT30U-F_1x02_P5.0mm_Vertical
- SW1: value (none) -> SW_DPDT_x2; footprint (none) -> Button_Switch_THT:SW_Slide_1P2T_CK_OS102011MS2Q
- U1: footprint (none) -> Mini360_step-down:Mini360_step-down
Connections:
- net GND: now also J6.1 (Pin_1); no longer J6.2 (Pin_2)
- net VCC: now also J6.2 (Pin_2); no longer J6.1 (Pin_1)
Changed lines of the file:
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@@
     (stroke (width 0) (type default) (color 0 0 0 0))
   )
-  (label "VCC" (at 54.102 57.404 0)
+  (label "VCC" (at 54.102 54.864 0)
     (effects (font (size 1.27 1.27)) (justify left bottom))
   )
@@
     (effects (font (size 1.27 1.27)) (justify left bottom))
   )
-  (label "GND" (at 54.102 54.864 0)
+  (label "GND" (at 54.102 57.404 0)
     (effects (font (size 1.27 1.27)) (justify left bottom))
   )
@@
       (effects (font (size 1.27 1.27)) (justify left))
     )
-    (property "Value" "" (id 1) (at 38.862 41.402 0)
-      (effects (font (size 1.27 1.27)) (justify left))
-    )
-    (property "Footprint" "" (id 2) (at 34.798 46.736 0)
+    (property "Value" "CENTRAL" (id 1) (at 38.862 41.402 0)
+      (effects (font (size 1.27 1.27)) (justify left))
+    )
+    (property "Footprint" "TerminalBlock:TerminalBlock_bornier-2_P5.08mm" (id 2) (at 34.798 46.736 0)
       (effects (font (size 1.27 1.27)) hide)
     )
@@
     (in_bom yes) (on_board yes) (fields_autoplaced)
     (property "Reference" "SW1" (id 0) (at 71.628 21.8272 0))
-    (property "Value" "" (id 1) (at 71.628 24.3641 0))
-    (property "Footprint" "" (id 2) (at 71.628 28.448 0)
+    (property "Value" "SW_DPDT_x2" (id 1) (at 71.628 24.3641 0))
+    (property "Footprint" "Button_Switch_THT:SW_Slide_1P2T_CK_OS102011MS2Q" (id 2) (at 71.628 28.448 0)
       (effects (font (size 1.27 1.27)) hide)
     )
@@
     (in_bom yes) (on_board yes)
     (property "Reference" "J5" (id 0) (at 49.022 39.37 0))
-    (property "Value" "" (id 1) (at 49.022 41.7631 0))
-    (property "Footprint" "" (id 2) (at 49.022 46.736 0)
+    (property "Value" "PISO" (id 1) (at 49.022 41.7631 0))
+    (property "Footprint" "TerminalBlock:TerminalBlock_bornier-2_P5.08mm" (id 2) (at 49.022 46.736 0)
       (effects (font (size 1.27 1.27)) hide)
     )
@@
     (in_bom yes) (on_board yes) (fields_autoplaced)
     (property "Reference" "J1" (id 0) (at 19.812 49.6402 0))
-    (property "Value" "" (id 1) (at 19.812 52.1771 0))
-    (property "Footprint" "" (id 2) (at 19.812 57.15 0)
+    (property "Value" "SENSORES" (id 1) (at 19.812 52.1771 0))
+    (property "Footprint" "TerminalBlock:TerminalBlock_bornier-2_P5.08mm" (id 2) (at 19.812 57.15 0)
       (effects (font (size 1.27 1.27)) hide)
     )
@@
       (effects (font (size 1.524 1.524)))
     )
-    (property "Footprint" "" (id 2) (at 36.83 28.702 0)
+    (property "Footprint" "Mini360_step-down:Mini360_step-down" (id 2) (at 36.83 28.702 0)
       (effects (font (size 1.524 1.524)) hide)
     )
@@
     (in_bom yes) (on_board yes) (fields_autoplaced)
     (property "Reference" "J3" (id 0) (at 34.544 49.8942 0))
-    (property "Value" "" (id 1) (at 34.544 52.4311 0))
-    (property "Footprint" "" (id 2) (at 34.544 57.404 0)
+    (property "Value" "BOTONES" (id 1) (at 34.544 52.4311 0))
+    (property "Footprint" "TerminalBlock:TerminalBlock_bornier-2_P5.08mm" (id 2) (at 34.544 57.404 0)
       (effects (font (size 1.27 1.27)) hide)
     )
@@
       (effects (font (size 1.27 1.27)) (justify left))
     )
-    (property "Value" "" (id 1) (at 52.832 52.07 0)
-      (effects (font (size 1.27 1.27)) (justify left))
-    )
-    (property "Footprint" "" (id 2) (at 49.022 57.404 0)
+    (property "Value" "BATERIA" (id 1) (at 52.832 52.07 0)
+      (effects (font (size 1.27 1.27)) (justify left))
+    )
+    (property "Footprint" "Connector_AMASS:AMASS_XT30U-F_1x02_P5.0mm_Vertical" (id 2) (at 49.022 57.404 0)
       (effects (font (size 1.27 1.27)) hide)
     )
@@
     (in_bom yes) (on_board yes)
     (property "Reference" "J2" (id 0) (at 20.066 39.2262 0))
-    (property "Value" "" (id 1) (at 20.066 41.402 0))
-    (property "Footprint" "" (id 2) (at 20.066 46.736 0)
-      (effects (font (size 1.27 1.27)) hide)
-    )
+    (property "Value" "MOTORES" (id 1) (at 20.066 41.402 0))
+    (property "Footprint" "Connector_AMASS:AMASS_XT30U-F_1x02_P5.0mm_Vertical" (id 2) (at 20.066 46.736 0)
+      (effects (font (size 1.27 1.27)) hide)
+    )
