File: placas/Sumo/alimentacion/THT/THT.kicad_pcb (KiCad board)
At the start: 2 copper layers, 40 x 44.2 mm, 11 parts, among them J1 SENSORES, J2 MOTORES, J3 BOTONES, J4 CENTRAL, J5 PISO, J6 BATERIA, SW1 SW_DPDT_x2, U1 Mini360

Commit message: wed
Connections:
- J6 pad 1: /VCC -> GND
- J6 pad 2: GND -> /VCC
Routing:
- net /VCC: track 36.3 -> 51.6 mm
- net GND: track 111.3 -> 109.9 mm
Changed lines of the file:
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@@
     (fp_line (start -2.6 -1.3) (end -0.9 -2.6) (layer "F.Fab") (width 0.1))
     (pad "1" thru_hole rect (at 0 0 180) (size 3.8 3.8) (drill 2.7) (layers *.Cu *.Mask)
-      (net 3 "/VCC") (pinfunction "Pin_1") (pintype "passive"))
+      (net 1 "GND") (pinfunction "Pin_1") (pintype "passive"))
     (pad "2" thru_hole circle (at 5 0 180) (size 4 4) (drill 2.7) (layers *.Cu *.Mask)
-      (net 1 "GND") (pinfunction "Pin_2") (pintype "passive"))
+      (net 3 "/VCC") (pinfunction "Pin_2") (pintype "passive"))
     (model "${KICAD6_3DMODEL_DIR}/Connector_AMASS.3dshapes/AMASS_XT30U-F_1x02_P5.0mm_Vertical.wrl"
       (offset (xyz 0 0 0))
@@
   (via (at 16.4592 89.7128) (size 3.5) (drill 3) (layers "F.Cu" "B.Cu") (free) (net 0))
   (via (at 49.7332 51.8668) (size 3.5) (drill 3) (layers "F.Cu" "B.Cu") (free) (net 0))
-  (segment (start 31.1804 82.256) (end 31.6484 81.788) (width 1) (layer "B.Cu") (net 1))
+  (segment (start 36.1804 83.3756) (end 34.5928 81.788) (width 1) (layer "B.Cu") (net 1))
   (segment (start 34.584 81.7968) (end 34.5928 81.788) (width 1) (layer "B.Cu") (net 1))
   (segment (start 43.7388 60.8076) (end 47.1424 60.8076) (width 1) (layer "B.Cu") (net 1))
@@
   (segment (start 47.0408 72.9888) (end 43.3432 72.9888) (width 1) (layer "B.Cu") (net 1))
   (segment (start 40.3332 60.8076) (end 43.7388 60.8076) (width 1) (layer "B.Cu") (net 1))
+  (segment (start 36.1804 88.4936) (end 36.1804 83.3756) (width 1) (layer "B.Cu") (net 1))
   (segment (start 22.4536 64.5668) (end 22.4536 65.2272) (width 1) (layer "B.Cu") (net 1))
-  (segment (start 31.1804 88.5444) (end 31.1804 82.256) (width 1) (layer "B.Cu") (net 1))
   (segment (start 22.352 64.4652) (end 22.4536 64.5668) (width 1) (layer "B.Cu") (net 1))
   (segment (start 47.1424 57.8104) (end 43.7388 54.4068) (width 1) (layer "B.Cu") (net 1))
   (segment (start 19.1008 64.4652) (end 22.352 64.4652) (width 1) (layer "B.Cu") (net 1))
+  (segment (start 36.1804 88.5444) (end 37.2872 88.5444) (width 1) (layer "B.Cu") (net 1))
   (segment (start 43.3432 72.9888) (end 34.5928 72.9888) (width 1) (layer "B.Cu") (net 1))
   (segment (start 18.9992 75.4888) (end 22.4536 75.4888) (width 1) (layer "B.Cu") (net 1))
-  (segment (start 31.6484 81.788) (end 34.5928 81.788) (width 1) (layer "B.Cu") (net 1))
   (segment (start 19.1516 53.4416) (end 22.4536 53.4416) (width 1) (layer "B.Cu") (net 1))
   (segment (start 35.306 62.5856) (end 35.2552 62.5348) (width 1) (layer "B.Cu") (net 2))
@@
   (segment (start 41.1988 56.4896) (end 41.1988 54.4068) (width 1) (layer "B.Cu") (net 2))
   (segment (start 35.2552 62.5348) (end 41.2496 56.5404) (width 1) (layer "B.Cu") (net 2))
-  (segment (start 39.624 86.2076) (end 39.624 81.28) (width 1) (layer "B.Cu") (net 3))
+  (segment (start 39.5224 92.0496) (end 39.5224 81.28) (width 1) (layer "B.Cu") (net 3))
   (segment (start 43.7496 81.28) (end 47.0408 77.9888) (width 1) (layer "B.Cu") (net 3))
+  (segment (start 39.624 81.28) (end 42.3672 81.28) (width 1) (layer "B.Cu") (net 3))
+  (segment (start 39.5224 81.28) (end 42.3672 81.28) (width 1) (layer "B.Cu") (net 3))
+  (segment (start 32.6136 92.0496) (end 39.5224 92.0496) (width 1) (layer "B.Cu") (net 3))
   (segment (start 47.0408 77.9888) (end 50.1288 77.9888) (width 1) (layer "B.Cu") (net 3))
   (segment (start 50.6476 77.47) (end 50.6476 67.2084) (width 1) (layer "B.Cu") (net 3))
+  (segment (start 31.1804 90.6164) (end 32.6136 92.0496) (width 1) (layer "B.Cu") (net 3))
   (segment (start 50.6476 67.2084) (end 49.3268 65.8876) (width 1) (layer "B.Cu") (net 3))
-  (segment (start 37.2872 88.5444) (end 39.624 86.2076) (width 1) (layer "B.Cu") (net 3))
-  (segment (start 39.624 81.28) (end 43.7496 81.28) (width 1) (layer "B.Cu") (net 3))
+  (segment (start 42.3672 81.28) (end 43.7496 81.28) (width 1) (layer "B.Cu") (net 3))
   (segment (start 50.1288 77.9888) (end 50.6476 77.47) (width 1) (layer "B.Cu") (net 3))
   (segment (start 49.3268 65.8876) (end 47.1424 65.8876) (width 1) (layer "B.Cu") (net 3))
-  (segment (start 36.1804 88.5444) (end 37.2872 88.5444) (width 1) (layer "B.Cu") (net 3))
+  (segment (start 31.1804 88.4936) (end 31.1804 90.6164) (width 1) (layer "B.Cu") (net 3))
   (segment (start 31.2436 70.7152) (end 31.2436 53.9423) (width 1) (layer "B.Cu") (net 4))
   (segment (start 31.75 71.2216) (end 31.2436 70.7152) (width 1) (layer "B.Cu") (net 4))
