File: placas/Sumo/piso/THT/Piso/Piso.kicad_pcb (KiCad board)
At the start: 2 copper layers, 28.7 x 34 mm, 6 parts, among them J1 Conn_01x04_Male, J2 Conn_01x04_Male, J3 Conn_01x04_Male, J4 Conn_01x04_Male, J5 Conn_01x04_Male, J6 Screw_Terminal_01x02

Commit message: wed
Routing:
- net /Vcc: track 102.8 -> 107.8 mm
- net GND: track 90.7 -> 91.5 mm
Other:
- board size 28.7 x 34 mm -> 30 x 34.8 mm
Changed lines of the file:
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@@
     )
   )
-  (gr_rect (start 52.07 28.956) (end 80.772 62.992) (layer "Edge.Cuts") (width 0.2) (fill none))
+  (gr_rect (start 51.308 28.6512) (end 81.3308 63.4492) (layer "Edge.Cuts") (width 0.2) (fill none))
   (gr_text "D\n" (at 72.39 42.672 180) (layer "F.SilkS")
     (effects (font (size 1 1) (thickness 0.25)) (justify mirror))
@@
   (via (at 54.102 60.96) (size 3.5) (drill 3) (layers "F.Cu" "B.Cu") (free) (net 0))
   (segment (start 53.086 29.972) (end 74.168 29.972) (width 1) (layer "B.Cu") (net 1))
-  (segment (start 75.946 61.468) (end 79.756 57.658) (width 1) (layer "B.Cu") (net 1))
+  (segment (start 56.953 56.124) (end 64.77 56.124) (width 1) (layer "B.Cu") (net 1))
   (segment (start 53.086 56.124) (end 53.086 40.386) (width 1) (layer "B.Cu") (net 1))
-  (segment (start 64.77 58.674) (end 67.564 61.468) (width 1) (layer "B.Cu") (net 1))
-  (segment (start 79.756 48.524) (end 76.143 48.524) (width 1) (layer "B.Cu") (net 1))
-  (segment (start 62.982 56.124) (end 64.77 57.912) (width 1) (layer "B.Cu") (net 1))
-  (segment (start 67.564 61.468) (end 75.946 61.468) (width 1) (layer "B.Cu") (net 1))
+  (segment (start 79.756 60.96) (end 79.756 48.524) (width 1) (layer "B.Cu") (net 1))
+  (segment (start 64.77 61.722) (end 78.994 61.722) (width 1) (layer "B.Cu") (net 1))
   (segment (start 56.953 42.662) (end 53.086 42.662) (width 1) (layer "B.Cu") (net 1))
   (segment (start 56.953 56.124) (end 53.086 56.124) (width 1) (layer "B.Cu") (net 1))
-  (segment (start 79.756 57.658) (end 79.756 48.524) (width 1) (layer "B.Cu") (net 1))
   (segment (start 74.168 29.972) (end 75.889 31.693) (width 1) (layer "B.Cu") (net 1))
-  (segment (start 64.77 57.912) (end 64.77 58.674) (width 1) (layer "B.Cu") (net 1))
+  (segment (start 64.77 56.124) (end 64.77 58.674) (width 1) (layer "B.Cu") (net 1))
+  (segment (start 79.756 48.524) (end 76.143 48.524) (width 1) (layer "B.Cu") (net 1))
+  (segment (start 78.994 61.722) (end 79.756 60.96) (width 1) (layer "B.Cu") (net 1))
   (segment (start 53.086 42.662) (end 53.086 40.386) (width 1) (layer "B.Cu") (net 1))
   (segment (start 53.086 40.386) (end 53.086 29.972) (width 1) (layer "B.Cu") (net 1))
   (segment (start 75.889 31.693) (end 75.889 35.062) (width 1) (layer "B.Cu") (net 1))
-  (segment (start 56.953 56.124) (end 62.982 56.124) (width 1) (layer "B.Cu") (net 1))
+  (segment (start 64.77 58.674) (end 64.77 61.722) (width 1) (layer "B.Cu") (net 1))
   (segment (start 54.864 31.75) (end 54.864 37.338) (width 1) (layer "B.Cu") (net 3))
   (segment (start 55.128 51.044) (end 56.953 51.044) (width 1) (layer "B.Cu") (net 3))
@@
   (segment (start 59.69 45.466) (end 55.88 45.466) (width 1) (layer "B.Cu") (net 3))
   (segment (start 69.85 58.674) (end 68.326 57.15) (width 1) (layer "B.Cu") (net 3))
+  (segment (start 69.85 58.674) (end 77.724 58.674) (width 1) (layer "B.Cu") (net 3))
   (segment (start 55.118 37.592) (end 55.128 37.582) (width 1) (layer "B.Cu") (net 3))
   (segment (start 70.866 31.75) (end 54.864 31.75) (width 1) (layer "B.Cu") (net 3))
-  (segment (start 78.222 53.604) (end 76.143 53.604) (width 1) (layer "B.Cu") (net 3))
-  (segment (start 69.85 58.674) (end 76.454 58.674) (width 1) (layer "B.Cu") (net 3))
   (segment (start 66.792 51.044) (end 56.953 51.044) (width 1) (layer "B.Cu") (net 3))
   (segment (start 74.432 40.142) (end 72.898 38.608) (width 1) (layer "B.Cu") (net 3))
   (segment (start 54.864 37.338) (end 55.118 37.592) (width 1) (layer "B.Cu") (net 3))
   (segment (start 68.326 52.578) (end 66.792 51.044) (width 1) (layer "B.Cu") (net 3))
-  (segment (start 78.232 56.896) (end 78.232 53.594) (width 1) (layer "B.Cu") (net 3))
+  (segment (start 78.232 58.166) (end 78.232 53.594) (width 1) (layer "B.Cu") (net 3))
   (segment (start 55.88 45.466) (end 55.118 46.228) (width 1) (layer "B.Cu") (net 3))
   (segment (start 68.326 57.15) (end 68.326 52.578) (width 1) (layer "B.Cu") (net 3))
   (segment (start 59.944 45.212) (end 59.69 45.466) (width 1) (layer "B.Cu") (net 3))
+  (segment (start 77.724 58.674) (end 78.232 58.166) (width 1) (layer "B.Cu") (net 3))
   (segment (start 59.68 37.582) (end 59.944 37.846) (width 1) (layer "B.Cu") (net 3))
-  (segment (start 76.454 58.674) (end 78.232 56.896) (width 1) (layer "B.Cu") (net 3))
   (segment (start 55.128 37.582) (end 56.953 37.582) (width 1) (layer "B.Cu") (net 3))
   (segment (start 55.118 51.034) (end 55.128 51.044) (width 1) (layer "B.Cu") (net 3))
@@
   (segment (start 72.898 33.782) (end 70.866 31.75) (width 1) (layer "B.Cu") (net 3))
   (segment (start 78.232 53.594) (end 78.222 53.604) (width 1) (layer "B.Cu") (net 3))
+  (segment (start 78.222 53.604) (end 76.143 53.604) (width 1) (layer "B.Cu") (net 3))
   (segment (start 56.953 37.582) (end 59.68 37.582) (width 1) (layer "B.Cu") (net 3))
   (segment (start 55.118 46.228) (end 55.118 51.034) (width 1) (layer "B.Cu") (net 3))
