File: placas/Sumo/piso/THT/Piso/Piso.kicad_sch (KiCad schematic)
At the start: 6 parts, among them J1 Conn_01x04_Male, J2 Conn_01x04_Male, J3 Conn_01x04_Male, J4 Conn_01x04_Male, J5 Conn_01x04_Male, J6 Screw_Terminal_01x02

Commit message: CAMBIOS
Other:
- moved on the sheet: J5, J6
Changed lines of the file:
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@@
     (effects (font (size 1.27 1.27)) (justify left bottom))
   )
-  (label "DATA4" (at 47.244 39.37 0)
+  (label "DATA4" (at 70.358 41.148 0)
     (effects (font (size 1.27 1.27)) (justify left bottom))
   )
-  (label "DATA3" (at 47.244 36.83 0)
+  (label "DATA3" (at 70.358 38.608 0)
     (effects (font (size 1.27 1.27)) (justify left bottom))
   )
@@
     (effects (font (size 1.27 1.27)) (justify left bottom))
   )
-  (label "DATA2" (at 47.244 34.29 0)
+  (label "DATA2" (at 70.358 36.068 0)
     (effects (font (size 1.27 1.27)) (justify left bottom))
   )
-  (label "Vcc" (at 48.26 20.574 0)
+  (label "Vcc" (at 71.374 22.352 0)
     (effects (font (size 1.27 1.27)) (justify left bottom))
   )
@@
     (effects (font (size 1.27 1.27)) (justify left bottom))
   )
-  (label "DATA1" (at 47.244 31.75 0)
+  (label "DATA1" (at 70.358 33.528 0)
     (effects (font (size 1.27 1.27)) (justify left bottom))
   )
@@
     (effects (font (size 1.27 1.27)) (justify left bottom))
   )
-  (symbol (lib_id "power:GND") (at 48.26 23.114 90) (unit 1)
+  (symbol (lib_id "power:GND") (at 71.374 24.892 90) (unit 1)
     (in_bom yes) (on_board yes) (fields_autoplaced)
-    (property "Reference" "#PWR?" (id 0) (at 54.61 23.114 0)
+    (property "Reference" "#PWR?" (id 0) (at 77.724 24.892 0)
       (effects (font (size 1.27 1.27)) hide)
     )
-    (property "Value" "GND" (id 1) (at 52.07 23.1139 90)
+    (property "Value" "GND" (id 1) (at 75.184 24.8919 90)
       (effects (font (size 1.27 1.27)) (justify right))
     )
-    (property "Footprint" "" (id 2) (at 48.26 23.114 0)
+    (property "Footprint" "" (id 2) (at 71.374 24.892 0)
       (effects (font (size 1.27 1.27)) hide)
     )
-    (property "Datasheet" "" (id 3) (at 48.26 23.114 0)
+    (property "Datasheet" "" (id 3) (at 71.374 24.892 0)
       (effects (font (size 1.27 1.27)) hide)
     )
@@
     (pin "4")
   )
-  (symbol (lib_id "Connector:Conn_01x04_Male") (at 42.164 34.29 0) (unit 1)
+  (symbol (lib_id "Connector:Conn_01x04_Male") (at 65.278 36.068 0) (unit 1)
     (in_bom yes) (on_board yes)
-    (property "Reference" "J5" (id 0) (at 46.228 26.416 0))
-    (property "Value" "Conn_01x04_Male" (id 1) (at 45.974 28.448 0))
-    (property "Footprint" "Connector_PinHeader_2.54mm:PinHeader_1x04_P2.54mm_Horizontal" (id 2) (at 42.164 34.29 0)
+    (property "Reference" "J5" (id 0) (at 69.342 28.194 0))
+    (property "Value" "Conn_01x04_Male" (id 1) (at 69.088 30.226 0))
+    (property "Footprint" "Connector_PinHeader_2.54mm:PinHeader_1x04_P2.54mm_Horizontal" (id 2) (at 65.278 36.068 0)
       (effects (font (size 1.27 1.27)) hide)
     )
-    (property "Datasheet" "~" (id 3) (at 42.164 34.29 0)
+    (property "Datasheet" "~" (id 3) (at 65.278 36.068 0)
       (effects (font (size 1.27 1.27)) hide)
     )
@@
     (pin "4")
   )
-  (symbol (lib_id "Connector:Screw_Terminal_01x02") (at 43.18 23.114 180) (unit 1)
+  (symbol (lib_id "Connector:Screw_Terminal_01x02") (at 66.294 24.892 180) (unit 1)
     (in_bom yes) (on_board yes) (fields_autoplaced)
-    (property "Reference" "J6" (id 0) (at 43.18 13.716 0))
-    (property "Value" "Screw_Terminal_01x02" (id 1) (at 43.18 16.256 0))
-    (property "Footprint" "TerminalBlock:TerminalBlock_bornier-2_P5.08mm" (id 2) (at 43.18 23.114 0)
+    (property "Reference" "J6" (id 0) (at 66.294 15.494 0))
+    (property "Value" "Screw_Terminal_01x02" (id 1) (at 66.294 18.034 0))
+    (property "Footprint" "TerminalBlock:TerminalBlock_bornier-2_P5.08mm" (id 2) (at 66.294 24.892 0)
       (effects (font (size 1.27 1.27)) hide)
     )
-    (property "Datasheet" "~" (id 3) (at 43.18 23.114 0)
+    (property "Datasheet" "~" (id 3) (at 66.294 24.892 0)
       (effects (font (size 1.27 1.27)) hide)
     )
