File: placas/Sumo/Motores/THT/THT/THT.kicad_sch (KiCad schematic)
At the start: 3 parts

Commit message: fgfgh
Parts:
- J1: renamed from J?; value Control Motores -> (none); footprint Connector_IDC:IDC-Header_2x04_P2.54mm_Vertical -> (none)
- gave numbers to parts that had none: 2
Changed lines of the file:
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@@
   (symbol (lib_id "Connector_Generic:Conn_02x04_Odd_Even") (at 68.834 54.864 0) (unit 1)
     (in_bom yes) (on_board yes) (fields_autoplaced)
-    (property "Reference" "J?" (id 0) (at 70.104 45.466 0))
-    (property "Value" "Control Motores" (id 1) (at 70.104 48.006 0))
-    (property "Footprint" "Connector_IDC:IDC-Header_2x04_P2.54mm_Vertical" (id 2) (at 68.834 54.864 0)
+    (property "Reference" "J1" (id 0) (at 70.104 45.466 0))
+    (property "Value" "" (id 1) (at 70.104 48.006 0))
+    (property "Footprint" "" (id 2) (at 68.834 54.864 0)
       (effects (font (size 1.27 1.27)) hide)
     )
@@
   (symbol (lib_id "MCU_Module:Arduino_UNO_R3") (at 37.592 46.228 0) (unit 1)
     (in_bom yes) (on_board yes) (fields_autoplaced)
-    (property "Reference" "A?" (id 0) (at 44.6914 19.6682 0)
+    (property "Reference" "A1" (id 0) (at 44.6914 19.6682 0)
       (effects (font (size 1.27 1.27)) (justify left))
     )
@@
   (symbol (lib_id "Connector:Conn_01x02_Male") (at 73.152 40.894 180) (unit 1)
     (in_bom yes) (on_board yes) (fields_autoplaced)
-    (property "Reference" "J?" (id 0) (at 73.8632 38.7893 0)
+    (property "Reference" "J2" (id 0) (at 73.8632 38.7893 0)
       (effects (font (size 1.27 1.27)) (justify right))
     )
@@
   (symbol_instances
     (path "/ca6d9730-64c7-44d0-8b63-c904e1f317bc"
-      (reference "A?") (unit 1) (value "Arduino_UNO_R3") (footprint "Module:Arduino_UNO_R3")
+      (reference "A1") (unit 1) (value "Arduino_UNO_R3") (footprint "Module:Arduino_UNO_R3")
     )
     (path "/8f07aa90-cd3b-43e7-87c6-9d611cdee86c"
-      (reference "J?") (unit 1) (value "Control Motores") (footprint "Connector_IDC:IDC-Header_2x04_P2.54mm_Vertical")
+      (reference "J1") (unit 1) (value "Control Motores") (footprint "Connector_IDC:IDC-Header_2x04_P2.54mm_Horizontal")
     )
     (path "/f07140d0-0a2c-4323-949d-ed33f8fdb4b9"
-      (reference "J?") (unit 1) (value "Conn_01x02_Male") (footprint "Connector_PinHeader_2.54mm:PinHeader_1x02_P2.54mm_Horizontal")
+      (reference "J2") (unit 1) (value "Conn_01x02_Male") (footprint "Connector_PinHeader_2.54mm:PinHeader_1x02_P2.54mm_Horizontal")
     )
   )
