File: placas/Sumo/Motores/THT/THT/THT.kicad_pcb (KiCad board)
At the start: 2 copper layers, 3 parts, among them J1 Control Motores, J2 Conn_01x02_Male

Commit message: fgfgh
Routing:
- net /PWM2: track 55.2 -> 53.7 mm
- net (no net): vias 0 -> 4
Other:
- board outline added: 69.7 x 54.7 mm
Changed lines of the file:
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@@
     )
   )
+  (gr_rect (start 20.9296 16.51) (end 90.678 71.2216) (layer "Edge.Cuts") (width 0.2) (fill none))
+  (via (at 23.114 69.1388) (size 3.5) (drill 3) (layers "F.Cu" "B.Cu") (free) (net 0))
+  (via (at 88.5444 18.4912) (size 3.5) (drill 3) (layers "F.Cu" "B.Cu") (free) (net 0))
+  (via (at 88.4936 69.0372) (size 3.5) (drill 3) (layers "F.Cu" "B.Cu") (free) (net 0))
+  (via (at 22.8092 18.6436) (size 3.5) (drill 3) (layers "F.Cu" "B.Cu") (free) (net 0))
   (segment (start 70.7644 41.8592) (end 66.1924 41.8592) (width 1) (layer "F.Cu") (net 9))
   (segment (start 66.1924 41.8592) (end 66.1416 41.8084) (width 1) (layer "F.Cu") (net 9))
@@
   (segment (start 71.201 67.7004) (end 71.201 45.2834) (width 1) (layer "B.Cu") (net 20))
   (segment (start 71.201 45.2834) (end 72.136 44.3484) (width 1) (layer "B.Cu") (net 20))
-  (segment (start 76.9541 44.3484) (end 86.4616 44.3484) (width 1) (layer "B.Cu") (net 21))
   (segment (start 68.661 68.8642) (end 68.661 67.7004) (width 1) (layer "B.Cu") (net 21))
+  (segment (start 76.9541 44.3484) (end 85.6996 44.3484) (width 1) (layer "B.Cu") (net 21))
+  (segment (start 85.6996 44.3484) (end 85.6996 70.4596) (width 1) (layer "B.Cu") (net 21))
   (segment (start 70.2564 70.4596) (end 68.661 68.8642) (width 1) (layer "B.Cu") (net 21))
-  (segment (start 86.4616 44.3484) (end 86.4616 70.4596) (width 1) (layer "B.Cu") (net 21))
-  (segment (start 86.4616 70.4596) (end 70.2564 70.4596) (width 1) (layer "B.Cu") (net 21))
+  (segment (start 85.6996 70.4596) (end 70.2564 70.4596) (width 1) (layer "B.Cu") (net 21))
   (segment (start 74.422 54.4068) (end 74.3712 54.4576) (width 1) (layer "F.Cu") (net 22))
   (segment (start 74.3712 54.4576) (end 66.1924 54.4576) (width 1) (layer "F.Cu") (net 22))

Commit message: CAMBIOS
Parts:
- A1: moved to B.Cu
- moved A1 14.2 mm to (62.5, 20.2), turned to 180 degrees
- moved J2 7.58 mm to (70.4, 26.6)
- moved J1 5.12 mm to (69.5, 40.8)
Routing:
- net /C2: track 9.63 -> 44.7 mm, vias 0 -> 2
- net /EN2: track 35.6 -> 69.9 mm
- net /C1: track 13.9 -> 44.4 mm, vias 0 -> 2
- net /PWM1: track 26.0 -> 52.4 mm
- net /EN1: track 32.8 -> 53.1 mm, vias 2 -> 0
- net /INB1: track 39.7 -> 59.9 mm
- net /INA1: track 29.0 -> 44.7 mm, vias 2 -> 0
- net /PWM2: track 53.7 -> 64.4 mm
- net /INA2: track 48.3 -> 58.4 mm
- net /INB2: track 37.9 -> 40.7 mm, vias 2 -> 0
- net (no net): vias 4 -> 0
Other:
- board size 69.7 x 54.7 mm -> 69.7 x 55.4 mm
