File: placas/Sumo/Placa conjunta/Placa conjunta.kicad_pcb (KiCad board)
At the start: 2 copper layers, 99.5 x 104.7 mm, 21 parts, among them J1 BATERIA1, J10 Conn_01x04_Male, J11 Conn_01x04_Male, J12 Conn_01x04_Male, J2 MOTORES, J3 Control Sensores, J6 Control Botones, J7 Conn_01x04_Male, J8 Conn_01x04_Male, J9 Conn_01x04_Male, SW1 SW_DPDT_x2, U1 YAAJ_BluePill_Part_Like_SWD_B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, U2 Mini360

Commit message: MAI
Parts:
- removed J12: Conn_01x04_Male, Connector_JST:JST_XH_B4B-XH-A_1x04_P2.50mm_Vertical
- added ?: , , F.Cu at (80.2, 38.0)
- added J3: Conn_01x02_Male, TerminalBlock:TerminalBlock_bornier-2_P5.08mm, F.Cu at (148.1, 42.7)
- J10: renamed from J11; footprint Connector_JST:JST_XH_B4B-XH-A_1x04_P2.50mm_Vertical -> Connector_PinSocket_2.54mm:PinSocket_1x04_P2.54mm_Vertical
- J4: renamed from J3; footprint Connector_IDC:IDC-Header_2x05_P2.54mm_Vertical -> Connector_IDC:IDC-Header_2x05_P2.54mm_Horizontal
- J6: renamed from J7; footprint Connector_JST:JST_XH_B4B-XH-A_1x04_P2.50mm_Vertical -> Connector_PinSocket_2.54mm:PinSocket_1x04_P2.54mm_Vertical
- J7: renamed from J8; footprint Connector_JST:JST_XH_B4B-XH-A_1x04_P2.50mm_Vertical -> Connector_PinSocket_2.54mm:PinSocket_1x04_P2.54mm_Vertical
- J8: renamed from J9; footprint Connector_JST:JST_XH_B4B-XH-A_1x04_P2.50mm_Vertical -> Connector_PinSocket_2.54mm:PinSocket_1x04_P2.54mm_Vertical
- J9: renamed from J10; footprint Connector_JST:JST_XH_B4B-XH-A_1x04_P2.50mm_Vertical -> Connector_PinSocket_2.54mm:PinSocket_1x04_P2.54mm_Vertical
- moved ? 17.1 mm to (148.1, 54.0)
- moved J9 8.31 mm to (55.7, 60.5), turned to 90 degrees
- moved J6 8.20 mm to (55.6, 85.8), turned to 90 degrees
- moved J10 8.09 mm to (55.7, 52.4), turned to 90 degrees
- moved J7 8.01 mm to (55.8, 77.5), turned to 90 degrees
- moved J8 7.93 mm to (55.7, 69.0), turned to 90 degrees
- renumbered J6 to J5
Connections:
- J4 pad 1: /5v -> /S4
- J4 pad 2: GND -> /S8
- J4 pad 3: /S4 -> /S3
- J4 pad 4: /S8 -> /S7
- J4 pad 5: /S3 -> /38khz
- J4 pad 6: /S7 -> /38khz
- U1 pad 25: /P6 -> /P5
- U1 pad 26: /P5 -> /P4
- U1 pad 27: /P4 -> /P3
- U1 pad 28: /P3 -> /P2
- U1 pad 29: /P2 -> /P1
- U1 pad 30: /P1 -> /EN1
- U1 pad 31: /EN1 -> /PWM1
- U1 pad 5: /PWM1 -> /S1
- U1 pad 6: /S1 -> /38khz
Routing:
- net GND: track 210.6 -> 304.7 mm
- net /5v: track 95.1 -> 151.8 mm, vias 2 -> 0
- net /P6: track 44.8 -> 0.00 mm
- net /3,3v: track 216.7 -> 188.8 mm, vias 0 -> 2
- net /38khz: track 0.00 -> 24.4 mm
- net /PWM1: track 61.2 -> 76.6 mm, vias 2 -> 0
- net /P4: track 54.6 -> 48.9 mm
- net /EN1: track 118.7 -> 122.7 mm, vias 2 -> 0
- net /P3: track 61.6 -> 57.6 mm
- net /P5: track 47.6 -> 44.7 mm
- net /S4: track 26.3 -> 28.8 mm
- net /S3: track 21.7 -> 24.1 mm
- net /S7: track 21.4 -> 23.8 mm
- net /P2: track 69.7 -> 67.6 mm
- net /P1: track 79.1 -> 77.1 mm
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Other:
- board size 99.5 x 104.7 mm -> 101.4 x 104.7 mm
