File: placas/Sumo/Placa conjunta/Placa conjunta.kicad_sch (KiCad schematic)
At the start: 18 parts, among them J1 BATERIA1, J10 Conn_01x04_Male, J11 Conn_01x04_Male, J12 Conn_01x04_Male, J2 MOTORES, J3 Control Sensores, J6 Control Botones, J7 Conn_01x04_Male, J8 Conn_01x04_Male, J9 Conn_01x04_Male, SW1 SW_DPDT_x2, U1 YAAJ_BluePill_Part_Like_SWD_B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, U2 Mini360

Commit message: MAI
Parts:
- removed J12: Conn_01x04_Male, Connector_JST:JST_XH_B4B-XH-A_1x04_P2.50mm_Vertical, symbol Connector:Conn_01x04_Male
- added J3: Conn_01x02_Male, TerminalBlock:TerminalBlock_bornier-2_P5.08mm, symbol Connector:Conn_01x02_Male
- J10: renamed from J11; footprint Connector_JST:JST_XH_B4B-XH-A_1x04_P2.50mm_Vertical -> (none)
- J4: renamed from J3; footprint Connector_IDC:IDC-Header_2x05_P2.54mm_Vertical -> Connector_IDC:IDC-Header_2x05_P2.54mm_Horizontal
- J6: renamed from J7; footprint Connector_JST:JST_XH_B4B-XH-A_1x04_P2.50mm_Vertical -> (none)
- J7: renamed from J8; footprint Connector_JST:JST_XH_B4B-XH-A_1x04_P2.50mm_Vertical -> (none)
- J8: renamed from J9; footprint Connector_JST:JST_XH_B4B-XH-A_1x04_P2.50mm_Vertical -> (none)
- J9: renamed from J10; footprint Connector_JST:JST_XH_B4B-XH-A_1x04_P2.50mm_Vertical -> (none)
- renumbered J6 to J5
Connections:
- net P6 is gone; now on net P5: U1.25 (PA0)
- net 5v: now also J3.1 (Pin_1); no longer J4.1 (Pin_1)
- net EN1: now also U1.30 (PA5); no longer U1.31 (PA6)
- net GND: now also J3.2 (Pin_2); no longer J4.2 (Pin_2)
- net P1: now also U1.29 (PA4); no longer U1.30 (PA5)
- net P2: now also U1.28 (PA3); no longer U1.29 (PA4)
- net P3: now also U1.27 (PA2); no longer U1.28 (PA3)
- net P4: now also U1.26 (PA1); no longer U1.27 (PA2)
- net P5: no longer U1.26 (PA1)
- net PWM1: now also U1.31 (PA6); no longer U1.5 (PA8)
- net S1: now also U1.5 (PA8); no longer U1.6 (PA9)
- net S3: now also J4.3 (Pin_3); no longer J4.5 (Pin_5)
- net S4: now also J4.1 (Pin_1); no longer J4.3 (Pin_3)
- net S7: now also J4.4 (Pin_4); no longer J4.6 (Pin_6)
- net S8: now also J4.2 (Pin_2); no longer J4.4 (Pin_4)
- new net 38khz: J4.5 (Pin_5), J4.6 (Pin_6), U1.6 (PA9)
- no-connect marks 11 -> 10
