File: placas/Sumo/sensores/THT/THT.kicad_pcb (KiCad board)
At the start: 2 copper layers, 37.1 x 56.6 mm, 11 parts, among them J3 Conn_01x02_Male, J6 Conn_02x04_Odd_Even, U1 Mini360

Commit message: fgdgf
Parts:
- removed J6: Conn_02x04_Odd_Even, Connector_IDC:IDC-Header_2x04_P2.54mm_Vertical
- added D3: DIODE, Diode_THT:D_5W_P12.70mm_Horizontal, F.Cu at (43.9, 60.6)
- added J2: Control Sensores, Connector_IDC:IDC-Header_2x05_P2.54mm_Vertical, F.Cu at (43.0, 22.4)
- moved J1 4.34 mm to (40.8, 67.1)
- moved U1 0.89 mm to (38.7, 48.7)
- renumbered D2 to D1, D3 to D2, D1 to D4, D4 to D5, D5 to D6, D8 to D7, D6 to D8, D7 to D9, J3 to J1
Connections:
- D1 pad 2: /gnd -> /data2
- D1 pad 3: /data2 -> /gnd
- D1 pad 4: unconnected-(D2-Pad4) -> /38Kh
- D2 pad 2: /gnd -> /data3
- D2 pad 3: /data3 -> /gnd
- D2 pad 4: unconnected-(D3-Pad4) -> /38Kh
- D4 pad 2: /gnd -> /data1
- D4 pad 3: /data1 -> /gnd
- D4 pad 4: unconnected-(D1-Pad4) -> /38Kh
- D5 pad 2: /gnd -> /data4
- D5 pad 3: /data4 -> /gnd
- D5 pad 4: unconnected-(D4-Pad4) -> /38Kh
- D6 pad 1: unconnected-(D5-Pad1) -> /38Kh
- D6 pad 2: /data5 -> /gnd
- D6 pad 3: /gnd -> /data5
- D7 pad 1: unconnected-(D8-Pad1) -> /38Kh
- D7 pad 2: /data8 -> /gnd
- D7 pad 3: /gnd -> /data8
- D8 pad 1: unconnected-(D6-Pad1) -> /38Kh
- D8 pad 2: /data6 -> /gnd
- D8 pad 3: /gnd -> /data6
- D9 pad 1: unconnected-(D7-Pad1) -> /38Kh
- D9 pad 2: /data7 -> /gnd
- D9 pad 3: /gnd -> /data7
- J1 pad 1: Net-(J3-Pad1) -> Net-(D3-Pad1)
- J1 pad 2: Net-(J3-Pad2) -> /gnd
- U1 pad 1: Net-(J3-Pad2) -> /gnd
- U1 pad 2: Net-(J3-Pad1) -> Net-(D3-Pad2)
Routing:
- net /38Kh: track 0.00 -> 156.8 mm
- net /gnd: track 0.00 -> 21.7 mm
- net Net-(D3-Pad2): track 0.00 -> 13.8 mm
- net Net-(D3-Pad1): track 0.00 -> 7.76 mm
- net Net-(J3-Pad2): track 7.44 -> 0.00 mm
- net Net-(J3-Pad1): track 7.44 -> 0.00 mm
- net /data1: track 24.3 -> 20.3 mm
- net /data8: track 42.7 -> 38.9 mm
- net /data5: track 24.1 -> 20.4 mm
- net /5v: track 199.8 -> 196.3 mm
- net /data4: track 43.3 -> 40.2 mm
- net /data3: track 30.0 -> 27.3 mm
- net /data7: track 29.8 -> 27.1 mm
- net /data2: track 27.9 -> 25.6 mm
- net /data6: track 27.8 -> 25.6 mm

Commit message: wed
Connections:
- J2 pad 6: unconnected-(J2-Pad6) -> /38Kh
Routing:
- net /gnd: track 21.7 -> 195.6 mm
- net /38Kh: track 156.8 -> 157.7 mm, vias 0 -> 1
- removed copper zone on F.Cu, net /gnd
Changed lines of the file:
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@@
   (net 12 "/38Kh")
   (net 13 "Net-(D3-Pad2)")
-  (net 14 "unconnected-(J2-Pad6)")
   (footprint "Connector_PinHeader_2.54mm:PinHeader_1x04_P2.54mm_Horizontal" (layer "F.Cu")
     (at 51.503 56.4)
@@
       (net 12 "/38Kh") (pinfunction "Pin_5") (pintype "passive"))
     (pad "6" thru_hole circle (at 2.54 5.08 270) (size 1.7 1.7) (drill 1) (layers *.Cu *.Mask)
-      (net 14 "unconnected-(J2-Pad6)") (pinfunction "Pin_6") (pintype "passive+no_connect"))
+      (net 12 "/38Kh") (pinfunction "Pin_6") (pintype "passive"))
     (pad "7" thru_hole circle (at 0 7.62 270) (size 1.7 1.7) (drill 1) (layers *.Cu *.Mask)
       (net 7 "/data5") (pinfunction "Pin_7") (pintype "passive"))
@@
   (segment (start 46.226 19.814) (end 46.226 33.784) (width 1) (layer "B.Cu") (net 1))
   (segment (start 42.9768 22.4123) (end 42.9768 19.9136) (width 1) (layer "B.Cu") (net 1))
+  (segment (start 28.5516 37.594) (end 28.5416 37.584) (width 1) (layer "F.Cu") (net 2))
+  (segment (start 27.5844 63.2968) (end 27.5844 56.388) (width 1) (layer "F.Cu") (net 2))
+  (segment (start 28.5416 40.5464) (end 28.5416 37.584) (width 1) (layer "F.Cu") (net 2))
+  (segment (start 28.6004 25.654) (end 28.6004 26.67) (width 1) (layer "F.Cu") (net 2))
+  (segment (start 48.006 61.3396) (end 48.006 49.5848) (width 1) (layer "F.Cu") (net 2))
+  (segment (start 34.1396 41.0972) (end 29.0924 41.0972) (width 1) (layer "F.Cu") (net 2))
+  (segment (start 27.5416 61.46) (end 27.5844 61.4172) (width 1) (layer "F.Cu") (net 2))
+  (segment (start 51.503 61.48) (end 48.1464 61.48) (width 1) (layer "F.Cu") (net 2))
+  (segment (start 27.5844 67.056) (end 35.7632 67.056) (width 1) (layer "F.Cu") (net 2))
+  (segment (start 24.439 49.522) (end 28.3544 49.522) (width 1) (layer "F.Cu") (net 2))
+  (segment (start 28.6004 17.5768) (end 28.6004 26.67) (width 1) (layer "F.Cu") (net 2))
+  (segment (start 49.022 17.1704) (end 29.0068 17.1704) (width 1) (layer "F.Cu") (net 2))
+  (segment (start 34.1396 56.3372) (end 28.6352 56.3372) (width 1) (layer "F.Cu") (net 2))
+  (segment (start 48.008 37.594) (end 28.5516 37.594) (width 1) (layer "F.Cu") (net 2))
+  (segment (start 28.6352 56.3372) (end 27.6352 56.3372) (width 1) (layer "F.Cu") (net 2))
+  (segment (start 48.006 37.592) (end 48.008 37.594) (width 1) (layer "F.Cu") (net 2))
+  (segment (start 49.022 25.5016) (end 49.022 17.1704) (width 1) (layer "F.Cu") (net 2))
+  (segment (start 51.503 25.656) (end 49.1764 25.656) (width 1) (layer "F.Cu") (net 2))
+  (segment (start 48.1464 61.48) (end 48.006 61.3396) (width 1) (layer "F.Cu") (net 2))
+  (segment (start 28.6352 56.3372) (end 28.5416 56.2436) (width 1) (layer "F.Cu") (net 2))
+  (segment (start 28.6004 37.6428) (end 28.5416 37.584) (width 1) (layer "F.Cu") (net 2))
+  (segment (start 29.0068 17.1704) (end 28.6004 17.5768) (width 1) (layer "F.Cu") (net 2))
+  (segment (start 27.6352 56.3372) (end 27.5844 56.388) (width 1) (layer "F.Cu") (net 2))
+  (segment (start 49.1764 25.656) (end 49.022 25.5016) (width 1) (layer "F.Cu") (net 2))
+  (segment (start 48.008 37.594) (end 51.503 37.594) (width 1) (layer "F.Cu") (net 2))
+  (segment (start 28.5924 25.646) (end 28.6004 25.654) (width 1) (layer "F.Cu") (net 2))
+  (segment (start 48.0588 49.532) (end 51.503 49.532) (width 1) (layer "F.Cu") (net 2))
+  (segment (start 24.439 61.46) (end 27.5416 61.46) (width 1) (layer "F.Cu") (net 2))
+  (segment (start 28.6004 26.67) (end 28.6004 37.6428) (width 1) (layer "F.Cu") (net 2))
+  (segment (start 48.006 49.5848) (end 48.0588 49.532) (width 1) (layer "F.Cu") (net 2))
+  (segment (start 28.5416 49.3348) (end 28.5416 40.5464) (width 1) (layer "F.Cu") (net 2))
+  (segment (start 27.5844 61.4172) (end 27.5844 67.056) (width 1) (layer "F.Cu") (net 2))
+  (segment (start 28.5416 56.2436) (end 28.5416 49.3348) (width 1) (layer "F.Cu") (net 2))
+  (segment (start 29.0924 41.0972) (end 28.5416 40.5464) (width 1) (layer "F.Cu") (net 2))
+  (segment (start 48.006 49.5848) (end 48.006 37.592) (width 1) (layer "F.Cu") (net 2))
+  (segment (start 24.439 25.646) (end 28.5924 25.646) (width 1) (layer "F.Cu") (net 2))
+  (segment (start 28.3544 49.522) (end 28.5416 49.3348) (width 1) (layer "F.Cu") (net 2))
+  (segment (start 28.5416 37.584) (end 24.439 37.584) (width 1) (layer "F.Cu") (net 2))
   (segment (start 32.8168 64.1096) (end 27.5844 64.1096) (width 1) (layer "B.Cu") (net 2))
   (segment (start 31.0896 56.3372) (end 34.1396 56.3372) (width 1) (layer "B.Cu") (net 2))
@@
   (segment (start 43.0276 34.29) (end 42.9768 34.2392) (width 1) (layer "B.Cu") (net 11))
   (segment (start 51.483 64) (end 51.503 64.02) (width 1) (layer "F.Cu") (net 12))
-  (segment (start 46.736 28.0964) (end 46.736 19.8628) (width 1) (layer "F.Cu") (net 12))
   (segment (start 51.503 64.02) (end 54.2664 64.02) (width 1) (layer "F.Cu") (net 12))
   (segment (start 54.7116 29.0576) (end 53.85 28.196) (width 1) (layer "F.Cu") (net 12))
   (segment (start 21.4964 40.124) (end 24.439 40.124) (width 1) (layer "F.Cu") (net 12))
-  (segment (start 37.9476 19.8628) (end 37.8968 19.9136) (width 1) (layer "F.Cu") (net 12))
+  (segment (start 51.503 28.196) (end 45.718 28.196) (width 1) (layer "F.Cu") (net 12))
+  (segment (start 26.7716 70.0024) (end 24.439 67.6698) (width 1) (layer "F.Cu") (net 12))
   (segment (start 21.4456 52.062) (end 24.439 52.062) (width 1) (layer "F.Cu") (net 12))
   (segment (start 54.6608 63.6256) (end 54.6608 52.07) (width 1) (layer "F.Cu") (net 12))
   (segment (start 54.2664 64.02) (end 54.6608 63.6256) (width 1) (layer "F.Cu") (net 12))
+  (segment (start 48.6664 70.0024) (end 26.7716 70.0024) (width 1) (layer "F.Cu") (net 12))
   (segment (start 21.836 64) (end 21.2344 63.3984) (width 1) (layer "F.Cu") (net 12))
   (segment (start 54.6588 52.072) (end 54.6588 40.4348) (width 1) (layer "F.Cu") (net 12))
+  (segment (start 45.3136 31.496) (end 45.6184 31.1912) (width 1) (layer "F.Cu") (net 12))
+  (segment (start 45.718 28.196) (end 45.6184 28.2956) (width 1) (layer "F.Cu") (net 12))
+  (segment (start 51.503 67.1658) (end 48.6664 70.0024) (width 1) (layer "F.Cu") (net 12))
+  (segment (start 21.2344 52.2732) (end 21.2344 40.386) (width 1) (layer "F.Cu") (net 12))
+  (segment (start 54.6588 40.4348) (end 54.7116 40.382) (width 1) (layer "F.Cu") (net 12))
+  (segment (start 37.8968 31.496) (end 45.3136 31.496) (width 1) (layer "F.Cu") (net 12))
+  (segment (start 45.6184 31.1912) (end 45.6184 28.2956) (width 1) (layer "F.Cu") (net 12))
   (segment (start 51.503 64.02) (end 51.503 67.1658) (width 1) (layer "F.Cu") (net 12))
-  (segment (start 21.2344 52.2732) (end 21.2344 40.386) (width 1) (layer "F.Cu") (net 12))
-  (segment (start 27.2796 70.5104) (end 24.439 67.6698) (width 1) (layer "F.Cu") (net 12))
-  (segment (start 54.6588 40.4348) (end 54.7116 40.382) (width 1) (layer "F.Cu") (net 12))
   (segment (start 54.6588 40.4348) (end 54.358 40.134) (width 1) (layer "F.Cu") (net 12))
-  (segment (start 46.736 19.8628) (end 37.9476 19.8628) (width 1) (layer "F.Cu") (net 12))
   (segment (start 54.358 40.134) (end 51.503 40.134) (width 1) (layer "F.Cu") (net 12))
   (segment (start 21.2344 52.2732) (end 21.4456 52.062) (width 1) (layer "F.Cu") (net 12))
@@
   (segment (start 22.0044 28.186) (end 24.439 28.186) (width 1) (layer "F.Cu") (net 12))
   (segment (start 54.6588 52.072) (end 51.503 52.072) (width 1) (layer "F.Cu") (net 12))
-  (segment (start 48.1584 70.5104) (end 27.2796 70.5104) (width 1) (layer "F.Cu") (net 12))
   (segment (start 24.439 64) (end 21.836 64) (width 1) (layer "F.Cu") (net 12))
   (segment (start 21.2344 63.3984) (end 21.2344 52.2732) (width 1) (layer "F.Cu") (net 12))
   (segment (start 21.2344 28.956) (end 22.0044 28.186) (width 1) (layer "F.Cu") (net 12))
-  (segment (start 51.503 67.1658) (end 48.1584 70.5104) (width 1) (layer "F.Cu") (net 12))
   (segment (start 54.7116 40.382) (end 54.7116 29.0576) (width 1) (layer "F.Cu") (net 12))
   (segment (start 21.2344 40.386) (end 21.2344 28.956) (width 1) (layer "F.Cu") (net 12))
-  (segment (start 37.8968 19.9136) (end 37.8968 22.4123) (width 1) (layer "F.Cu") (net 12))
-  (segment (start 51.503 28.196) (end 46.8356 28.196) (width 1) (layer "F.Cu") (net 12))
+  (segment (start 24.439 67.6698) (end 24.439 64) (width 1) (layer "F.Cu") (net 12))
   (segment (start 53.85 28.196) (end 51.503 28.196) (width 1) (layer "F.Cu") (net 12))
-  (segment (start 24.439 67.6698) (end 24.439 64) (width 1) (layer "F.Cu") (net 12))
-  (segment (start 46.8356 28.196) (end 46.736 28.0964) (width 1) (layer "F.Cu") (net 12))
   (segment (start 54.6608 52.07) (end 54.6588 52.072) (width 1) (layer "F.Cu") (net 12))
+  (via (at 37.8968 31.496) (size 0.8) (drill 0.4) (layers "F.Cu" "B.Cu") (net 12))
+  (segment (start 37.8968 24.9523) (end 37.8968 22.4123) (width 1) (layer "B.Cu") (net 12))
+  (segment (start 37.8968 24.9523) (end 37.8968 31.496) (width 1) (layer "B.Cu") (net 12))
   (segment (start 40.1828 56.3372) (end 43.2796 56.3372) (width 1) (layer "B.Cu") (net 13))
   (segment (start 35.9664 60.5536) (end 40.1828 56.3372) (width 1) (layer "B.Cu") (net 13))
   (segment (start 31.1912 60.5536) (end 35.9664 60.5536) (width 1) (layer "B.Cu") (net 13))
-  (zone (net 2) (net_name "/gnd") (layer "F.Cu") (hatch edge 0.508)
-    (connect_pads (clearance 1))
-    (min_thickness 0.254) (filled_areas_thickness no)
-    (fill yes (thermal_gap 0.508) (thermal_bridge_width 0.508))
-    (polygon
-      (pts
-        (xy 56.386 71.122)
-        (xy 19.81 71.122)
-        (xy 19.81 14.988)
-        (xy 56.386 14.988)
-      )
-    )
-  )
 )

Commit message: fhfhfhg
Routing:
- net /gnd: track 195.6 -> 181.8 mm
Changed lines of the file:
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@@
   (segment (start 27.5416 61.46) (end 27.5844 61.4172) (width 1) (layer "F.Cu") (net 2))
   (segment (start 51.503 61.48) (end 48.1464 61.48) (width 1) (layer "F.Cu") (net 2))
-  (segment (start 27.5844 67.056) (end 35.7632 67.056) (width 1) (layer "F.Cu") (net 2))
   (segment (start 24.439 49.522) (end 28.3544 49.522) (width 1) (layer "F.Cu") (net 2))
   (segment (start 28.6004 17.5768) (end 28.6004 26.67) (width 1) (layer "F.Cu") (net 2))
@@
   (segment (start 48.006 49.5848) (end 48.0588 49.532) (width 1) (layer "F.Cu") (net 2))
   (segment (start 28.5416 49.3348) (end 28.5416 40.5464) (width 1) (layer "F.Cu") (net 2))
-  (segment (start 27.5844 61.4172) (end 27.5844 67.056) (width 1) (layer "F.Cu") (net 2))
   (segment (start 28.5416 56.2436) (end 28.5416 49.3348) (width 1) (layer "F.Cu") (net 2))
   (segment (start 29.0924 41.0972) (end 28.5416 40.5464) (width 1) (layer "F.Cu") (net 2))

Commit message: fgfgh
Routing:
- net /gnd: track 181.8 -> 179.9 mm
Changed lines of the file:
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@@
   (segment (start 42.9768 22.4123) (end 42.9768 19.9136) (width 1) (layer "B.Cu") (net 1))
   (segment (start 28.5516 37.594) (end 28.5416 37.584) (width 1) (layer "F.Cu") (net 2))
-  (segment (start 27.5844 63.2968) (end 27.5844 56.388) (width 1) (layer "F.Cu") (net 2))
   (segment (start 28.5416 40.5464) (end 28.5416 37.584) (width 1) (layer "F.Cu") (net 2))
+  (segment (start 27.6352 56.3372) (end 28.6352 56.3372) (width 1) (layer "F.Cu") (net 2))
   (segment (start 28.6004 25.654) (end 28.6004 26.67) (width 1) (layer "F.Cu") (net 2))
   (segment (start 48.006 61.3396) (end 48.006 49.5848) (width 1) (layer "F.Cu") (net 2))
+  (segment (start 27.5844 56.388) (end 27.6352 56.3372) (width 1) (layer "F.Cu") (net 2))
   (segment (start 34.1396 41.0972) (end 29.0924 41.0972) (width 1) (layer "F.Cu") (net 2))
   (segment (start 27.5416 61.46) (end 27.5844 61.4172) (width 1) (layer "F.Cu") (net 2))
@@
   (segment (start 34.1396 56.3372) (end 28.6352 56.3372) (width 1) (layer "F.Cu") (net 2))
   (segment (start 48.008 37.594) (end 28.5516 37.594) (width 1) (layer "F.Cu") (net 2))
-  (segment (start 28.6352 56.3372) (end 27.6352 56.3372) (width 1) (layer "F.Cu") (net 2))
   (segment (start 48.006 37.592) (end 48.008 37.594) (width 1) (layer "F.Cu") (net 2))
   (segment (start 49.022 25.5016) (end 49.022 17.1704) (width 1) (layer "F.Cu") (net 2))
@@
   (segment (start 28.6352 56.3372) (end 28.5416 56.2436) (width 1) (layer "F.Cu") (net 2))
   (segment (start 28.6004 37.6428) (end 28.5416 37.584) (width 1) (layer "F.Cu") (net 2))
+  (segment (start 27.5844 61.4172) (end 27.5844 56.388) (width 1) (layer "F.Cu") (net 2))
   (segment (start 29.0068 17.1704) (end 28.6004 17.5768) (width 1) (layer "F.Cu") (net 2))
-  (segment (start 27.6352 56.3372) (end 27.5844 56.388) (width 1) (layer "F.Cu") (net 2))
   (segment (start 49.1764 25.656) (end 49.022 25.5016) (width 1) (layer "F.Cu") (net 2))
   (segment (start 48.008 37.594) (end 51.503 37.594) (width 1) (layer "F.Cu") (net 2))
@@
   (segment (start 53.85 28.196) (end 51.503 28.196) (width 1) (layer "F.Cu") (net 12))
   (segment (start 54.6608 52.07) (end 54.6588 52.072) (width 1) (layer "F.Cu") (net 12))
-  (via (at 37.8968 31.496) (size 0.8) (drill 0.4) (layers "F.Cu" "B.Cu") (net 12))
+  (via (at 37.8968 31.496) (size 1.8) (drill 1) (layers "F.Cu" "B.Cu") (net 12))
   (segment (start 37.8968 24.9523) (end 37.8968 22.4123) (width 1) (layer "B.Cu") (net 12))
   (segment (start 37.8968 24.9523) (end 37.8968 31.496) (width 1) (layer "B.Cu") (net 12))

Commit message: MAI
Parts:
- removed the D3 at (43.9, 60.6)
- removed D9: Conn_01x04_Male, Connector_PinHeader_2.54mm:PinHeader_1x04_P2.54mm_Horizontal
- removed U1: Mini360, Mini360_step-down:Mini360_step-down
- added D5: Conn_01x04_Male, Connector_PinHeader_2.54mm:PinHeader_1x04_P2.54mm_Vertical, F.Cu at (29.2, 38.9)
- added REF**: MountingHole_2.7mm_Pad, MountingHole:MountingHole_2.7mm_Pad, F.Cu at (21.5, 46.1)
- added REF**: MountingHole_2.7mm_Pad, MountingHole:MountingHole_2.7mm_Pad, F.Cu at (56.6, 17.2)
- D1, D2, D6, D7, D8: footprint Connector_PinHeader_2.54mm:PinHeader_1x04_P2.54mm_Horizontal -> Connector_PinHeader_2.54mm:PinHeader_1x04_P2.54mm_Vertical
- D3: renamed from D4; footprint Connector_PinHeader_2.54mm:PinHeader_1x04_P2.54mm_Horizontal -> Connector_PinHeader_2.54mm:PinHeader_1x04_P2.54mm_Vertical
- D4: renamed from D5; footprint Connector_PinHeader_2.54mm:PinHeader_1x04_P2.54mm_Horizontal -> Connector_PinHeader_2.54mm:PinHeader_1x04_P2.54mm_Vertical
- moved J1 50.3 mm to (23.5, 19.8), turned to 0 degrees
- moved D7 31.7 mm to (48.5, 43.4), turned to -90 degrees
- moved D3 26.4 mm to (29.2, 34.6), turned to 90 degrees
- moved D8 24.1 mm to (48.5, 38.9), turned to -90 degrees
- moved D1 22.5 mm to (29.2, 30.1), turned to 90 degrees
- moved D4 22.0 mm to (48.5, 34.6), turned to -90 degrees
- moved D6 15.9 mm to (29.2, 43.4), turned to 90 degrees
- moved D2 14.7 mm to (48.4, 30.1), turned to -90 degrees
- moved J2 4.44 mm to (38.6, 22.0), turned to 90 degrees
Connections:
- D6 pad 1: /38Kh -> /5v
- D6 pad 2: /gnd -> /data6
- D6 pad 3: /data5 -> /gnd
- D6 pad 4: /5v -> /38Kh
- D7 pad 1: /38Kh -> /5v
- D7 pad 2: /gnd -> /data7
- D7 pad 3: /data8 -> /gnd
- D7 pad 4: /5v -> /38Kh
- D8 pad 1: /38Kh -> /5v
- D8 pad 2: /gnd -> /data8
- D8 pad 3: /data6 -> /gnd
- D8 pad 4: /5v -> /38Kh
- J1 pad 1: Net-(D3-Pad1) -> /5v
- J2 pad 1: /data2 -> /data1
- J2 pad 10: /data7 -> /data8
- J2 pad 2: /data3 -> /data5
- J2 pad 3: /data1 -> /data2
- J2 pad 4: /data4 -> /data6
- J2 pad 7: /data5 -> /data3
- J2 pad 8: /data8 -> /data7
- J2 pad 9: /data6 -> /data4
Routing:
- net /38Kh: track 157.7 -> 54.6 mm, vias 1 -> 0
- net /5v: track 196.3 -> 133.3 mm, vias 0 -> 14
- net /gnd: track 179.9 -> 117.2 mm
- net /data6: track 25.6 -> 54.0 mm
- net /data5: track 20.4 -> 42.4 mm
- net /data7: track 27.1 -> 48.1 mm
- net /data3: track 27.3 -> 8.22 mm
- net /data4: track 40.2 -> 25.1 mm
- net Net-(D3-Pad2): track 13.8 -> 0.00 mm
- net /data1: track 20.3 -> 32.9 mm
- net /data2: track 25.6 -> 15.7 mm
- net Net-(D3-Pad1): track 7.76 -> 0.00 mm
- net /data8: track 38.9 -> 34.6 mm
- net (no net): vias 4 -> 0
Other:
- board size 37.1 x 56.6 mm -> 39.5 x 33.3 mm
- board text removed: "5v"
- board text removed: "DATOS"
- board text removed: "GND"
- board text removed: "VCC"
