File: placas/Sumo/sensores/THT/THT.kicad_sch (KiCad schematic)
At the start: 12 parts, among them J1 Conn_01x02_Male, J2 Conn_02x04_Odd_Even, U1 Mini360

Commit message: yho
Parts:
- removed J2: Conn_02x04_Odd_Even, Connector_IDC:IDC-Header_2x04_P2.54mm_Vertical, symbol Connector_Generic:Conn_02x04_Odd_Even
- added J2: Control Sensores, Connector_IDC:IDC-Header_2x05_P2.54mm_Vertical, symbol Connector_Generic:Conn_02x05_Odd_Even
Connections:
- net 38Kh: now also J2.5 (Pin_5)
- net data1: now also J2.3 (Pin_3)
- net data2: now also J2.1 (Pin_1)
- net data3: now also J2.2 (Pin_2)
- net data4: now also J2.4 (Pin_4)
- net data5: now also J2.7 (Pin_7)
- net data6: now also J2.9 (Pin_9)
- net data7: now also J2.10 (Pin_10)
- net data8: now also J2.8 (Pin_8)
- no-connect marks 0 -> 1
Changed lines of the file:
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@@
 (kicad_sch (version 20211123) (generator eeschema)
   (paper "A4")
+  (no_connect (at 123.444 52.578))
   (wire (pts (xy 55.372 47.498) (xy 58.674 47.498))
     (stroke (width 0) (type default) (color 0 0 0 0))
@@
     (effects (font (size 1.27 1.27)) (justify right bottom))
   )
+  (label "data1" (at 110.744 50.038 180)
+    (effects (font (size 1.27 1.27)) (justify right bottom))
+  )
   (label "5v" (at 134.874 27.686 270)
     (effects (font (size 1.27 1.27)) (justify right bottom))
@@
     (effects (font (size 1.27 1.27)) (justify right bottom))
   )
-  (label "data8" (at 97.282 53.848 0)
-    (effects (font (size 1.27 1.27)) (justify left bottom))
-  )
   (label "5v" (at 115.57 27.686 270)
     (effects (font (size 1.27 1.27)) (justify right bottom))
@@
     (effects (font (size 1.27 1.27)) (justify right bottom))
   )
+  (label "data4" (at 123.444 50.038 0)
+    (effects (font (size 1.27 1.27)) (justify left bottom))
+  )
   (label "data6" (at 137.414 27.686 270)
     (effects (font (size 1.27 1.27)) (justify right bottom))
@@
     (effects (font (size 1.27 1.27)) (justify right bottom))
   )
-  (label "data3" (at 97.282 48.768 0)
+  (label "data7" (at 123.444 57.658 0)
     (effects (font (size 1.27 1.27)) (justify left bottom))
   )
@@
     (effects (font (size 1.27 1.27)) (justify right bottom))
   )
-  (label "data4" (at 97.282 51.308 0)
-    (effects (font (size 1.27 1.27)) (justify left bottom))
+  (label "data2" (at 110.744 47.498 180)
+    (effects (font (size 1.27 1.27)) (justify right bottom))
   )
   (label "gnd" (at 17.272 44.958 180)
     (effects (font (size 1.27 1.27)) (justify right bottom))
   )
-  (label "data5" (at 84.582 53.848 180)
-    (effects (font (size 1.27 1.27)) (justify right bottom))
-  )
   (label "gnd" (at 47.752 44.958 90)
     (effects (font (size 1.27 1.27)) (justify left bottom))
@@
     (effects (font (size 1.27 1.27)) (justify right bottom))
   )
+  (label "data6" (at 110.744 57.658 180)
+    (effects (font (size 1.27 1.27)) (justify right bottom))
+  )
+  (label "data8" (at 123.444 55.118 0)
+    (effects (font (size 1.27 1.27)) (justify left bottom))
+  )
   (label "gnd" (at 39.37 26.416 270)
     (effects (font (size 1.27 1.27)) (justify right bottom))
@@
     (effects (font (size 1.27 1.27)) (justify right bottom))
   )
-  (label "data7" (at 97.282 56.388 0)
-    (effects (font (size 1.27 1.27)) (justify left bottom))
+  (label "data5" (at 110.744 55.118 180)
+    (effects (font (size 1.27 1.27)) (justify right bottom))
   )
   (label "data7" (at 155.448 27.94 270)
@@
     (effects (font (size 1.27 1.27)) (justify right bottom))
   )
+  (label "38Kh" (at 110.744 52.578 180)
+    (effects (font (size 1.27 1.27)) (justify right bottom))
+  )
   (label "gnd" (at 120.65 27.686 270)
     (effects (font (size 1.27 1.27)) (justify right bottom))
@@
     (effects (font (size 1.27 1.27)) (justify right bottom))
   )
-  (label "data6" (at 84.582 56.388 180)
-    (effects (font (size 1.27 1.27)) (justify right bottom))
-  )
   (label "gnd" (at 76.962 27.686 270)
     (effects (font (size 1.27 1.27)) (justify right bottom))
@@
     (effects (font (size 1.27 1.27)) (justify right bottom))
   )
-  (label "data2" (at 84.582 48.768 180)
-    (effects (font (size 1.27 1.27)) (justify right bottom))
-  )
   (label "38Kh" (at 36.83 26.416 270)
     (effects (font (size 1.27 1.27)) (justify right bottom))
   )
-  (label "data1" (at 84.582 51.308 180)
-    (effects (font (size 1.27 1.27)) (justify right bottom))
-  )
   (label "data2" (at 22.098 26.924 270)
     (effects (font (size 1.27 1.27)) (justify right bottom))
@@
   (label "5v" (at 152.908 27.94 270)
     (effects (font (size 1.27 1.27)) (justify right bottom))
+  )
+  (label "data3" (at 123.444 47.498 0)
+    (effects (font (size 1.27 1.27)) (justify left bottom))
   )
   (label "38Kh" (at 123.19 27.686 270)
@@
     (pin "4")
   )
-  (symbol (lib_id "Connector_Generic:Conn_02x04_Odd_Even") (at 89.662 51.308 0) (unit 1)
-    (in_bom yes) (on_board yes) (fields_autoplaced)
-    (property "Reference" "J2" (id 0) (at 90.932 41.91 0))
-    (property "Value" "Conn_02x04_Odd_Even" (id 1) (at 90.932 44.45 0))
-    (property "Footprint" "Connector_IDC:IDC-Header_2x04_P2.54mm_Vertical" (id 2) (at 89.662 51.308 0)
-      (effects (font (size 1.27 1.27)) hide)
-    )
-    (property "Datasheet" "~" (id 3) (at 89.662 51.308 0)
-      (effects (font (size 1.27 1.27)) hide)
-    )
-    (pin "1")
+  (symbol (lib_id "Connector:Conn_01x04_Male") (at 157.988 22.86 270) (unit 1)
+    (in_bom yes) (on_board yes) (fields_autoplaced)
+    (property "Reference" "D9" (id 0) (at 156.718 17.78 90))
+    (property "Value" "Conn_01x04_Male" (id 1) (at 156.718 20.32 90))
+    (property "Footprint" "Connector_PinHeader_2.54mm:PinHeader_1x04_P2.54mm_Horizontal" (id 2) (at 157.988 22.86 0)
+      (effects (font (size 1.27 1.27)) hide)
+    )
+    (property "Datasheet" "~" (id 3) (at 157.988 22.86 0)
+      (effects (font (size 1.27 1.27)) hide)
+    )
+    (pin "1")
+    (pin "2")
+    (pin "3")
+    (pin "4")
+  )
+  (symbol (lib_id "Connector_Generic:Conn_02x05_Odd_Even") (at 115.824 52.578 0) (unit 1)
+    (in_bom yes) (on_board yes)
+    (property "Reference" "J2" (id 0) (at 117.094 42.5282 0))
+    (property "Value" "Control Sensores" (id 1) (at 117.348 44.196 0))
+    (property "Footprint" "Connector_IDC:IDC-Header_2x05_P2.54mm_Vertical" (id 2) (at 115.824 52.578 0)
+      (effects (font (size 1.27 1.27)) hide)
+    )
+    (property "Datasheet" "~" (id 3) (at 115.824 52.578 0)
+      (effects (font (size 1.27 1.27)) hide)
+    )
+    (pin "1")
+    (pin "10")
     (pin "2")
     (pin "3")
@@
     (pin "7")
     (pin "8")
-  )
-  (symbol (lib_id "Connector:Conn_01x04_Male") (at 157.988 22.86 270) (unit 1)
-    (in_bom yes) (on_board yes) (fields_autoplaced)
-    (property "Reference" "D9" (id 0) (at 156.718 17.78 90))
-    (property "Value" "Conn_01x04_Male" (id 1) (at 156.718 20.32 90))
-    (property "Footprint" "Connector_PinHeader_2.54mm:PinHeader_1x04_P2.54mm_Horizontal" (id 2) (at 157.988 22.86 0)
-      (effects (font (size 1.27 1.27)) hide)
-    )
-    (property "Datasheet" "~" (id 3) (at 157.988 22.86 0)
-      (effects (font (size 1.27 1.27)) hide)
-    )
-    (pin "1")
-    (pin "2")
-    (pin "3")
-    (pin "4")
+    (pin "9")
   )
   (symbol (lib_id "mini360:Mini360") (at 32.512 47.498 180) (unit 1)
@@
       (reference "J1") (unit 1) (value "Conn_01x02_Male") (footprint "TerminalBlock:TerminalBlock_bornier-2_P5.08mm")
     )
-    (path "/9e39e8aa-f617-428a-954b-c9bfeec97fe2"
-      (reference "J2") (unit 1) (value "Conn_02x04_Odd_Even") (footprint "Connector_IDC:IDC-Header_2x04_P2.54mm_Vertical")
+    (path "/a306aa16-bd62-4213-9f7e-930339d076aa"
+      (reference "J2") (unit 1) (value "Control Sensores") (footprint "Connector_IDC:IDC-Header_2x05_P2.54mm_Vertical")
     )
     (path "/c6c62f17-6c47-4c80-9bd1-90dbd52adf9d"

Commit message: wed
Connections:
- net 38Kh: now also J2.6 (Pin_6)
- no-connect marks 1 -> 0
Changed lines of the file:
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@@
 (kicad_sch (version 20211123) (generator eeschema)
   (paper "A4")
-  (no_connect (at 123.444 52.578))
   (wire (pts (xy 55.372 47.498) (xy 58.674 47.498))
     (stroke (width 0) (type default) (color 0 0 0 0))
@@
     (effects (font (size 1.27 1.27)) (justify right bottom))
   )
+  (label "38Kh" (at 123.444 52.578 0)
+    (effects (font (size 1.27 1.27)) (justify left bottom))
+  )
   (label "data4" (at 123.444 50.038 0)

Commit message: MAI
Parts:
- removed D3: DIODE, Diode_THT:D_5W_P12.70mm_Horizontal, symbol Simulation_SPICE:DIODE
- removed D9: Conn_01x04_Male, Connector_PinHeader_2.54mm:PinHeader_1x04_P2.54mm_Horizontal, symbol Connector:Conn_01x04_Male
- removed U1: Mini360, Mini360_step-down:Mini360_step-down, symbol mini360:Mini360
- added D5: Conn_01x04_Male, Connector_PinHeader_2.54mm:PinHeader_1x04_P2.54mm_Vertical, symbol Connector:Conn_01x04_Male
- D1, D2: footprint Connector_PinHeader_2.54mm:PinHeader_1x04_P2.54mm_Horizontal -> (none)
- D3: renamed from D4; footprint Connector_PinHeader_2.54mm:PinHeader_1x04_P2.54mm_Horizontal -> (none)
- D4: renamed from D5; footprint Connector_PinHeader_2.54mm:PinHeader_1x04_P2.54mm_Horizontal -> (none)
- D6, D7, D8: footprint Connector_PinHeader_2.54mm:PinHeader_1x04_P2.54mm_Horizontal -> Connector_PinHeader_2.54mm:PinHeader_1x04_P2.54mm_Vertical
Connections:
- net 38Kh: now also D6.4 (Pin_4), D7.4 (Pin_4), D8.4 (Pin_4), D5.4 (Pin_4); no longer D6.1 (Pin_1), D7.1 (Pin_1), D8.1 (Pin_1)
- net 5v: now also D6.1 (Pin_1), D7.1 (Pin_1), D8.1 (Pin_1), J1.1 (Pin_1), D5.1 (Pin_1); no longer D6.4 (Pin_4), D7.4 (Pin_4), D8.4 (Pin_4)
- net data1: now also J2.1 (Pin_1); no longer J2.3 (Pin_3)
- net data2: now also J2.3 (Pin_3); no longer J2.1 (Pin_1)
- net data3: now also J2.7 (Pin_7); no longer J2.2 (Pin_2)
- net data4: now also J2.9 (Pin_9); no longer J2.4 (Pin_4)
- net data5: now also J2.2 (Pin_2), D5.2 (Pin_2); no longer D6.3 (Pin_3), J2.7 (Pin_7)
- net data6: now also D6.2 (Pin_2), J2.4 (Pin_4); no longer D8.3 (Pin_3), J2.9 (Pin_9)
- net data7: now also D7.2 (Pin_2), J2.8 (Pin_8); no longer J2.10 (Pin_10)
- net data8: now also D8.2 (Pin_2), J2.10 (Pin_10); no longer D7.3 (Pin_3), J2.8 (Pin_8)
- net gnd: now also D6.3 (Pin_3), D7.3 (Pin_3), D8.3 (Pin_3), D5.3 (Pin_3); no longer D6.2 (Pin_2), D7.2 (Pin_2), D8.2 (Pin_2)
Other:
- moved on the sheet: J1, J2
