File: placas/Sumo/Placa conjunta/V1/Placa conjunta.kicad_pcb (KiCad board)
At the start: 2 copper layers, 101.4 x 104.7 mm, 22 parts, among them J1 BATERIA1, J10 Conn_01x04_Male, J2 MOTORES, J3 Conn_01x02_Male, J4 Control Sensores, J5 Control Botones, J6 Conn_01x04_Male, J7 Conn_01x04_Male, J8 Conn_01x04_Male, J9 Conn_01x04_Male, SW1 SW_DPDT_x2, U1 YAAJ_BluePill_Part_Like_SWD_B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, U2 Mini360

Commit message: dfg
Parts:
- D1, D3: value DIODE -> type="D" model="DIODE" lib=""
