File: placas/Laberinto/Nano/MISA NANO/MISA NANO.kicad_pcb (KiCad board)
At the start: 2 copper layers, 78.1 x 66.1 mm, 27 parts, among them J1 Conn_01x06_Female, J2 Conn_01x06_Female, J3 Conn_01x04_Male, J4 Conn_01x04_Male, J5 Conn_01x04_Male, J6 Conn_01x04_Male, J7 Conn_01x08_Female, J8 Conn_01x02_Male, SW1 SW_Push, SW2 SW_Push, SW4 SW_DPDT_x2, U1 Mt3608, U3 L293

Commit message: gfgf
Changed lines of the file:
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@@
   (segment (start 124.67 57.9) (end 115.99 57.9) (width 1) (layer "F.Cu") (net 4))
   (segment (start 137.83 58) (end 137.8 57.97) (width 0.8) (layer "F.Cu") (net 4))
-  (segment (start 106.66 68.32) (end 106.71 68.37) (width 0.8) (layer "F.Cu") (net 4))
+  (segment (start 113.13 68.37) (end 106.71 68.37) (width 0.8) (layer "F.Cu") (net 4))
   (segment (start 135.1 60.455) (end 127.48 60.455) (width 1) (layer "F.Cu") (net 4))
-  (segment (start 106.71 68.37) (end 113.13 68.37) (width 0.8) (layer "F.Cu") (net 4))
   (segment (start 143.41 58) (end 137.83 58) (width 0.8) (layer "F.Cu") (net 4))
+  (segment (start 106.71 68.37) (end 106.66 68.32) (width 0.8) (layer "F.Cu") (net 4))
   (via (at 115.57 58.32) (size 1.8) (drill 1) (layers "F.Cu" "B.Cu") (net 4))
   (via (at 113.13 68.37) (size 1.8) (drill 1) (layers "F.Cu" "B.Cu") (net 4))
