File: placas/miniSumo/Jarrones/PP sense/V2/pp sense/pp sense.kicad_sch (KiCad schematic)
At the start: 39 parts, among them J2 Conn_01x06_Pin, Q1 BC547, Q2 BC547, Q3 BC547, Q4 BC547, U1 LM339

Commit message: gfgf
Parts:
- removed D10: IR RECEIVER, LED_THT:LED_D5.0mm, symbol Device:LED
- removed D11, D8: INDICADOR, LED_SMD:LED_1206_3216Metric_Pad1.42x1.75mm_HandSolder, symbol Device:LED
- removed D12: IR TRANSMITTER, LED_THT:LED_D5.0mm, symbol Device:LED
- removed Q1, Q2, Q3, Q4: BC547, Package_TO_SOT_THT:TO-92_Inline, symbol Transistor_BJT:BC547
- removed R10, R14: 47k, Resistor_SMD:R_1206_3216Metric_Pad1.30x1.75mm_HandSolder, symbol Device:R
- removed R11, R13, R15, R20, R9: 1k, Resistor_SMD:R_1206_3216Metric_Pad1.30x1.75mm_HandSolder, symbol Device:R
- removed R12: 100, Resistor_SMD:R_1206_3216Metric_Pad1.30x1.75mm_HandSolder, symbol Device:R
- D2: value INDICADOR -> IR TRANSMITTER; footprint LED_SMD:LED_1206_3216Metric_Pad1.42x1.75mm_HandSolder -> LED_THT:LED_D5.0mm
- D3: value IR TRANSMITTER -> IR RECEIVER
- D4: value IR RECEIVER -> IR TRANSMITTER
- D5: value INDICADOR -> IR RECEIVER; footprint LED_SMD:LED_1206_3216Metric_Pad1.42x1.75mm_HandSolder -> LED_THT:LED_D5.0mm
- R1, R5, R7: value 1k -> 10k; footprint Resistor_SMD:R_1206_3216Metric_Pad1.30x1.75mm_HandSolder -> Resistor_THT:R_Axial_DIN0411_L9.9mm_D3.6mm_P5.08mm_Vertical
- R2: value 47k -> 10k; footprint Resistor_SMD:R_1206_3216Metric_Pad1.30x1.75mm_HandSolder -> Resistor_THT:R_Axial_DIN0411_L9.9mm_D3.6mm_P5.08mm_Vertical
- R6: value 47k -> 100
Connections:
- net +5V: now also D1.1 (K), D3.1 (K), D5.1 (K), D7.1 (K), R16.1, R4.1, R6.1, R8.1
- net D1: now also D7.2 (A), R1.1, U1.7 (+); no longer U1.5 (+)
- net D2: now also D1.2 (A), R2.1, U1.5 (+); no longer R5.1, U1.7 (+)
- net D3: now also D3.2 (A), R5.1
- net D4: now also D5.2 (A), R7.1; no longer R1.1
- net GND: now also D2.2 (A), D4.2 (A), D6.2 (A), D9.2 (A), R1.2, R2.2, R5.2, R7.2; no longer D2.1 (K), D5.1 (K), R16.1, R2.1, R4.1, R6.1, R8.1
- net at R18.1, U1.1: now also J2.4 (Pin_4); no longer J2.3 (Pin_3)
- net at R17.1, U1.13: now also J2.1 (Pin_1); no longer J2.2 (Pin_2)
- net at R4.2: now also D2.1 (K); no longer D3.1 (K)
- net at R6.2: now also D4.1 (K); no longer R7.1
- net at R19.1, U1.2: now also J2.3 (Pin_3); no longer J2.4 (Pin_4)
- net at R3.1, U1.14: now also J2.2 (Pin_2); no longer J2.1 (Pin_1)
- removed net VCC: D1.1 (K), D3.2 (A), D4.1 (K), D6.2 (A), D7.1 (K), D9.2 (A)
Other:
- moved on the sheet: D7
