File: placas/miniSumo/Jarrones/PP sense/V2/pp sense/pp sense.kicad_pcb (KiCad board)
At the start: 2 copper layers, 97.5 x 29.6 mm, 23 parts, among them J2 Conn_01x06_Pin, U1 LM339

Commit message: fngvfng
Routing:
- net Net-(J2-Pin_1): track 40.4 -> 52.7 mm
- net /D4: track 44.4 -> 50.8 mm
- net +5V: track 208.8 -> 204.1 mm
- net Net-(U1A--): track 36.5 -> 40.2 mm
