File: placas/miniSumo/Sifones/placa central/V1/placa central.kicad_pcb (KiCad board)
At the start: 2 copper layers, 91.9 x 40.9 mm, 29 parts, among them J1 Screw_Terminal_01x02, J10 Conn_01x04_Male, J2 Conn_01x02_Socket, J3 Conn_01x02_Socket, J4 Conn_01x04_Male, J5 Conn_01x04_Male, J6 Conn_01x04_Male, J9 Conn_01x04_Male, SW1 SW_DPDT_x2, SW3 SW_Push, SW4 SW_Push, U1 L293, U2 Mt3608

Commit message: gfgf
Routing:
- net GND: track 303.9 -> 304.6 mm
- net /SHARP_D: track 18.8 -> 18.2 mm
