File: placas/miniSumo/sensores/Msense 555 prueba/msense_prueba/msense_prueba.kicad_pcb (KiCad board)
At the start: 2 copper layers, 98 x 70.1 mm, 22 parts, among them J1 Conn_01x05_Pin, Q1 BC547, U1 LM555xM, U2 TSOP17xx, U3 TSOP17xx, U4 TSOP17xx

Commit message: vbv
Other:
- board size 98 x 70.1 mm -> 81.8 x 39.4 mm
Changed lines of the file:
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@@
     )
   )
-  (gr_rect (start 37.846 21.082) (end 135.89 91.186)
+  (gr_rect (start 46.228 21.082) (end 128.016 60.452)
     (stroke (width 0.2) (type default)) (fill none) (layer "Edge.Cuts"))
   (segment (start 67.056 50.292) (end 62.778 50.292) (width 0.5) (layer "B.Cu") (net 1))
